File: HW-MAPLE-Med/mapleCUx_med_010.brd (EAGLE design)
At the start: 82.6 x 50 mm, 37 parts, among them IC31 ATMEGA168-TQFP, X1 SMA, X2 SMA, X3 SMA, X31 M03X2, X4 SMA

Commit message: Medium Test1
Parts:
- removed C3: 22pF, rcl:C0805
- removed CC4: CC1101_MODULE1SMD, wireless:CC1101_MODULE1_SMD
- removed CC_X1, CC_X2, CC_X4: (no value), con-lstb:MA05-2
- removed CTX-DB: 1365-10, con-leotronics:1365-10
- removed NRF24L01+: NRF24L01+, diy-modules:WIRELESS-NRF24L01
- removed U$1: W5100_LAN_MODULE, lan:W5100_LAN_MODULE
- removed U$3: CC1101_MODULE3_DIL, wireless:CC1101_MODULE3_DIL
- removed U$6: NRF24L01+SMD, wireless:NRF24L01+SMD
- added CC2-EXT: CC1101_MODULE3_DIL, wireless:CC1101_MODULE3_DIL
- added CC3: CC1101_MODULE1SMD, wireless:CC1101_MODULE1_SMD
- added MYSENS: NRF24L01+SMD, wireless:NRF24L01+SMD
- C7: value 4,7 -> 4,7uF
- moved LED32 104.6 mm to (67.9, 48.3)
- moved R32 102.4 mm to (67.9, 46.4), flipped to the bottom, turned to 180 degrees
- moved CC_X0 100.3 mm to (49.5, 43.2)
- moved UART1 78.0 mm to (59.7, 47.0), turned to 0 degrees
- moved C7 77.8 mm to (48.3, 17.1), flipped to the bottom, turned to 90 degrees
- moved R34 73.8 mm to (37.5, 33.0), flipped to the bottom
- moved C5 73.1 mm to (54.6, 38.1)
- moved C32 73.0 mm to (37.5, 36.2), flipped to the bottom, turned to 180 degrees
- moved X31 72.3 mm to (49.5, 24.1), turned to 180 degrees
- moved U$2 68.7 mm to (2.54, 2.54), turned to 90 degrees
- moved C6 68.7 mm to (50.8, 31.8)
- moved UART0 68.4 mm to (59.7, 43.2), turned to 0 degrees
- moved IC31 66.0 mm to (36.8, 44.5), flipped to the bottom
- moved C31 64.5 mm to (33.7, 31.1), flipped to the bottom, turned to 90 degrees
- moved X4 62.6 mm to (82.5, 23.5)
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Connections:
- removed net MOSI2: U$1.5
- removed net N$8: CTX-DB.7
- removed net NC: CTX-DB.9
- net +5V: no longer U$1.1
- net CC_CS1: no longer CC_X1.7
- net CC_CS2: now also CC2-EXT.CSN; no longer CC_X2.7
- net CC_CS3: now also CC3.CSN; no longer CC4.CSN, CC_X4.7
- net CC_IN_1: no longer CC_X1.6
- net CC_IN_2: now also CC2-EXT.GDO2; no longer CC_X2.6
- net CC_IN_3: now also CC3.GDO2; no longer CC4.GDO2, CC_X4.6
- net CC_OUT_1: no longer CC_X1.8
- net CC_OUT_2: now also CC2-EXT.GDO0; no longer CC_X2.8
- net CE-A: now also MYSENS.CE; no longer NRF24L01+.3
- net CSN-A: now also MYSENS.CSN; no longer NRF24L01+.4
- net GND: now also C7.2, CC2-EXT.GND@0, CC2-EXT.GND@1, CC3.GND@0, CC3.GND@1, CC3.GND@2, MYSENS.GND; no longer C3.1, C7.1, CC4.GND@0, CC4.GND@1, CC4.GND@2, CC_X1.10, CC_X1.9, CC_X2.10, CC_X2.9, CC_X4.10, CC_X4.9, CTX-DB.3, CTX-DB.5, NRF24L01+.1, U$1.2, U$1.7, U$3.GND@0, U$3.GND@1, U$6.GND
- net IRQ-A: now also MYSENS.IRQ; no longer NRF24L01+.8
- net M-SCK: now also MYSENS.SCK; no longer NRF24L01+.5
- net MISO-A: now also MYSENS.MISO; no longer NRF24L01+.7
- net MISO1: now also CC2-EXT.MISO, CC3.MISO; no longer CC4.MISO, CC_X1.5, CC_X2.5, CC_X4.5
- net MISO2: no longer U$1.8
- net MOSI-A: now also MYSENS.MOSI; no longer NRF24L01+.6
- net MOSI1: now also CC2-EXT.MOSI, CC3.MOSI; no longer CC4.MOSI, CC_X1.3, CC_X2.3, CC_X4.3
- net N$2: now also CC3.ANT; no longer CC4.ANT
- net NRESET: no longer CTX-DB.10
- net SCK1: now also CC2-EXT.SCK, CC3.SCLK; no longer CC4.SCLK, CC_X1.4, CC_X2.4, CC_X4.4
- net SCK2: no longer U$1.6
- net SWCLK/TCK: no longer CTX-DB.4
- net SWDIO/TMS: no longer CTX-DB.2
- net SWO/TDO: no longer CTX-DB.6
- net TDI: no longer CTX-DB.8
- net VCC: now also C7.1, CC2-EXT.VCC@0, CC2-EXT.VCC@1, CC3.VCC, MYSENS.VCC; no longer C3.2, C7.2, CC4.VCC, CC_X1.1, CC_X1.2, CC_X2.1, CC_X2.2, CC_X4.1, CC_X4.2, CTX-DB.1, NRF24L01+.2, U$3.VCC@0, U$3.VCC@1, U$6.VCC
- net WIZ_CS: no longer U$1.3
- net WIZ_RST: no longer U$1.4
Routing:
- net GND: track 0.00 -> 459.8 mm, vias 0 -> 2
- net VCC: track 0.00 -> 210.8 mm, vias 0 -> 1
- net MISO1: track 0.00 -> 116.8 mm, vias 0 -> 2
- net SCK1: track 0.00 -> 99.9 mm, vias 0 -> 3
- net RX-MAPLE: track 0.00 -> 95.3 mm, vias 0 -> 1
- net MISO-A: track 0.00 -> 87.0 mm, vias 0 -> 1
- net MOSI1: track 0.00 -> 85.2 mm, vias 0 -> 3
- net MOSI-A: track 0.00 -> 75.8 mm, vias 0 -> 1
- net +5V: track 0.00 -> 75.5 mm
- net TX_DBG: track 0.00 -> 68.3 mm
- net M-SCK: track 0.00 -> 63.7 mm, vias 0 -> 1
- net RX_DBG: track 0.00 -> 62.9 mm
- net CC_OUT_0: track 0.00 -> 61.0 mm
- net M-RES: track 0.00 -> 59.1 mm, vias 0 -> 2
- net CC_IN_0: track 0.00 -> 56.1 mm
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Other:
- board size 82.6 x 50 mm -> 82.7 x 50.2 mm
