File: HW-MAPLE-Med/mapleCUx_med_010.sch (EAGLE design)
At the start: 35 parts, among them IC31 ATMEGA168-TQFP, X1 SMA, X2 SMA, X3 SMA, X31 M03X2, X4 SMA

Commit message: Medium Test1
Parts:
- removed C3: 22pF, rcl:C-EUC0805
- removed CC_X1, CC_X2, CC_X4, W5500NIREN: (no value), con-lstb:MA05-2
- removed CTX-DB: 1365-10, con-leotronics:1365-10
- removed NRF24L01+: NRF24L01+, diy-modules:WIRELESS-NRF24L01
- removed U$1: MAPLEMINI, maplemini-small:MAPLEMINI
- removed U$3: CC1101_MODULE3_DIL, wireless:CC1101_MODULE3_DIL
- removed W5100: (no value), con-lsta:FE05-2
- added CC2-EXT: CC1101_MODULE3_DIL, wireless:CC1101_MODULE3_DIL
- added MYSENS: NRF24L01+SMD, wireless:NRF24L01+SMD
- added U$2: W5500_LAN_MODULE, lan:W5500_LAN_MODULE
- added U$4: MAPLEMINI, maplemini-mall:MAPLEMINI
- added U$5: HM-MOD-UARTDIL, wireless:HM-MOD-UARTDIL
- C7: value 4,7 -> 4,7uF
- renumbered CC4 to CC3
Connections:
- removed net N$8: CTX-DB-7.S
- removed net NC: CTX-DB-9.S
- net +5V: now also U$2.1, U$4.VIN; no longer U$1.VIN, W5100.1, W5500NIREN.1
- net CC_CS0: now also U$4.7/AIN/SPI1_SS; no longer U$1.7/AIN/SPI1_SS
- net CC_CS1: now also U$4.12; no longer CC_X1.7, U$1.12
- net CC_CS2: now also CC2-EXT.CSN, U$4.15/PWM/I2C1_SDA; no longer CC_X2.7, U$1.15/PWM/I2C1_SDA
- net CC_CS3: now also U$4.3/PWM/AIN; no longer CC_X4.7, U$1.3/PWM/AIN
- net CC_IN_0: now also U$4.11/PWM/AIN; no longer U$1.11/PWM/AIN
- net CC_IN_1: now also U$4.18; no longer CC_X1.6, U$1.18
- net CC_IN_2: now also CC2-EXT.GDO2, U$4.16/PWM/I2C1_SCL; no longer CC_X2.6, U$1.16/PWM/I2C1_SCL
- net CC_IN_3: now also U$4.14; no longer CC_X4.6, U$1.14
- net CC_OUT_0: now also U$4.10/PWM/AIN; no longer U$1.10/PWM/AIN
- net CC_OUT_1: now also U$4.17; no longer CC_X1.8, U$1.17
- net CC_OUT_2: now also CC2-EXT.GDO0, U$4.13; no longer CC_X2.8, U$1.13
- net CE-A: now also MYSENS.CE; no longer NRF24L01+.CE
- net CSN-A: now also MYSENS.CSN; no longer NRF24L01+.CSN
- net GND: now also C7.2, CC2-EXT.GND@0, CC2-EXT.GND@1, MYSENS.GND, U$2.3, U$4.2/BOOT1, U$4.AV-; no longer C3.1, C7.1, CC_X1.10, CC_X1.9, CC_X2.10, CC_X2.9, CC_X4.10, CC_X4.9, CTX-DB-3.S, CTX-DB-5.S, NRF24L01+.GND, U$1.2/BOOT1, U$1.AV-, W5100.2, W5100.7, W5500NIREN.3
- net IRQ-A: now also MYSENS.IRQ; no longer NRF24L01+.IRQ
- net M-SCK: now also MYSENS.SCK; no longer NRF24L01+.SCK
- net MISO-A: now also MYSENS.MISO; no longer NRF24L01+.MISO
- net MISO1: now also CC2-EXT.MISO, U$4.5/PWM/AIN/SPI1_MISO; no longer CC_X1.5, CC_X2.5, CC_X4.5, U$1.5/PWM/AIN/SPI1_MISO
- net MISO2: now also U$2.4, U$4.29/SPI2_MISO; no longer U$1.29/SPI2_MISO, W5100.8, W5500NIREN.4
- net MOSI-A: now also MYSENS.MOSI; no longer NRF24L01+.MOSI
- net MOSI1: now also CC2-EXT.MOSI, U$4.4/PWM/AIN/SPI1_MOSI; no longer CC_X1.3, CC_X2.3, CC_X4.3, U$1.4/PWM/AIN/SPI1_MOSI
- net NRESET: now also U$4.RESET; no longer CTX-DB-10.S, U$1.RESET
- net RST: now also U$2.6, U$4.28/SPI2_MOSI; no longer U$1.28/SPI2_MOSI, W5100.5, W5500NIREN.6
- net RX-MAPLE: now also U$4.8/PWM/AIN/RX2; no longer U$1.8/PWM/AIN/RX2
- net RX1: now also U$4.0/RX3/I2C2_SDA; no longer U$1.0/RX3/I2C2_SDA
- net RX_DBG: now also U$4.25/PWM/RX1; no longer U$1.25/PWM/RX1
- net SCK1: now also CC2-EXT.SCLK, U$4.6/AIN/SPI1_SCK; no longer CC_X1.4, CC_X2.4, CC_X4.4, U$1.6/AIN/SPI1_SCK
- net SCK2: now also U$2.10, U$4.30/SPI2_SCK; no longer U$1.30/SPI2_SCK, W5100.6, W5500NIREN.10
- net SWCLK/TCK: now also U$4.21; no longer CTX-DB-4.S, U$1.21
- net SWDIO/TMS: now also U$4.22; no longer CTX-DB-2.S, U$1.22
- net SWO/TDO: now also U$4.19; no longer CTX-DB-6.S, U$1.19
- net TDI: now also U$4.20; no longer CTX-DB-8.S, U$1.20
- net TX-MAPLE: now also U$4.9/PWM/AIN/TX2; no longer U$1.9/PWM/AIN/TX2
- net TX1: now also U$4.1/TX3/I2C2_SCL; no longer U$1.1/TX3/I2C2_SCL
- net TX_DBG: now also U$4.26/PWM/TX1; no longer U$1.26/PWM/TX1
- net VCC: now also C7.1, CC2-EXT.VCC@0, CC2-EXT.VCC@1, MYSENS.VCC, U$4.AV+; no longer C3.2, C7.2, CC_X1.1, CC_X1.2, CC_X2.1, CC_X2.2, CC_X4.1, CC_X4.2, CTX-DB-1.S, NRF24L01+.VCC, U$1.AV+
- net WIZ_CS: now also U$2.8, U$4.31/SPI2_SS; no longer U$1.31/SPI2_SS, W5100.3, W5500NIREN.8
- net WIZ_RST: now also U$2.5, U$4.27/PWM; no longer U$1.27/PWM, W5100.4, W5500NIREN.5
Other:
- moved on the sheet: C7
