File: HW-MAPLE-Med/mapleCUx_med_018.sch (EAGLE design)
At the start: 30 parts, among them IC31 ATMEGA168-TQFP, X1 SMA, X2 SMA, X3 SMA, X31 M03X2, X4 SMA

Commit message: Medium-Version Draft
Parts:
- removed CC3: CC1101_MODULE1SMD, wireless:CC1101_MODULE1SMD
- removed CC_X0: (no value), con-lstb:MA05-2
- removed U$2: W5500_LAN_MODULE, lan:W5500_LAN_MODULE
- removed U$5: HM-MOD-UARTDIL, wireless:HM-MOD-UARTDIL
- removed X4: SMA, sma:SMA
- added C3: 22pF, rcl:C-EUC0805
- added CC2-EXT1: CC1101_MODULE3_DIL, wireless:CC1101_MODULE3_DIL
- added CC4: CC1101_MODULE1SMD, wireless:CC1101_MODULE1SMD
- added HMMOD-UART: HM-MOD-UARTDIL, wireless:HM-MOD-UARTDIL
- added IC2: LAN-USR-ES1, Martin-Communication:LAN-USR-ES1
- added X5: (no value), adafruit:SMACONNECTOR_EDGE_UFL
- CC0: value CC1101_MODULE1SMD -> CC1101
- X1, X2, X3: value SMA -> (none); device sma:SMA -> adafruit:SMACONNECTOR_EDGE_UFL
Connections:
- new net N$33: IC2.!INT!
- net +5V: no longer U$2.1
- net CC_CS0: now also CC2-EXT1.CSN; no longer CC_X0.7
- net CC_CS3: now also CC4.CSN; no longer CC3.CSN
- net CC_IN_0: now also CC2-EXT1.GDO2; no longer CC_X0.6
- net CC_IN_3: now also CC4.GDO2; no longer CC3.GDO2
- net CC_OUT_0: now also CC2-EXT1.GDO0; no longer CC_X0.8
- net GND: now also C3.1, CC2-EXT1.GND@0, CC2-EXT1.GND@1, CC4.GND@1, CC4.GND@2, CC4.GND@3, HMMOD-UART.GND, IC2.GND, IC2.GND@1, IC2.GND@2, U$4.GND, X1.GND1, X1.GND2, X1.GND3, X1.GND4, X2.GND1, X2.GND2, X2.GND3, X2.GND4, X3.GND1, X3.GND2, X3.GND3, X3.GND4, X5.GND1, X5.GND2, X5.GND3, X5.GND4; no longer CC3.GND@1, CC3.GND@2, CC3.GND@3, CC_X0.10, CC_X0.9, U$2.3, X1.2, X1.3, X1.4, X1.5, X2.2, X2.3, X2.4, X2.5, X3.2, X3.3, X3.4, X3.5, X4.2, X4.3, X4.4, X4.5
- net MISO1: now also CC2-EXT1.MISO, CC4.MISO; no longer CC3.MISO, CC_X0.5
- net MISO2: now also IC2.MISO; no longer U$2.4
- net MOSI1: now also CC2-EXT1.MOSI, CC4.MOSI; no longer CC3.MOSI, CC_X0.3
- net N$1: now also CC1.ANT, X1.ANT; no longer CC2.ANT, X3.1
- net N$2: now also CC4.ANT, X3.ANT; no longer CC3.ANT, X4.1
- net N$3: now also CC2.ANT, X2.ANT; no longer CC1.ANT, X1.1
- net N$4: now also X5.ANT; no longer X2.1
- net RST: now also IC2.MOSI; no longer U$2.6
- net RX-MAPLE: now also HMMOD-UART.TX
- net SCK1: now also CC2-EXT1.SCLK, CC4.SCLK; no longer CC3.SCLK, CC_X0.4
- net SCK2: now also IC2.SCLK; no longer U$2.10
- net TX-MAPLE: now also HMMOD-UART.RX
- net VCC: now also C3.2, CC2-EXT1.VCC@0, CC2-EXT1.VCC@1, CC4.VCC, HMMOD-UART.VCC, IC2.V+, IC2.V+@1, U$4.VCC; no longer CC3.VCC, CC_X0.1, CC_X0.2
- net WIZ_CS: now also IC2.!SCS!; no longer U$2.8
- net WIZ_RST: now also IC2.RES; no longer U$2.5
Other:
- note added: "HomeMatic"
- note added: "LAN"
- note added: "MySensors"
- note added: "Transceiver 866 / 433 MHz"
- note removed: "W5500 NiRen 55x28mm Drill dist 23,1mm"
- moved on the sheet: C1, C2, C31, C32, C4, C5, C6, C7, CC0, CC1, CC2, CC2-EXT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
