File: HW-MAPLE-Med/mapleCUx_med_024.sch (EAGLE design)
At the start: 31 parts, among them IC2 LAN-USR-ES1, IC31 ATMEGA168-TQFP, X31 M03X2

Commit message: 1.2 Large - more docu
Parts:
- removed CC2-EXT1: CC1101_MODULE3_DIL, wireless:CC1101_MODULE3_DIL
- removed IC2: LAN-USR-ES1, Martin-Communication:LAN-USR-ES1
- removed X2: (no value), adafruit:SMACONNECTOR_EDGE_UFL
- added ANT2: TPPAD1-13, testpad:TPPAD1-13
Connections:
- removed net N$33: IC2.!INT!
- net CC_CS0: no longer CC2-EXT1.CSN
- net CC_IN_0: no longer CC2-EXT1.GDO2
- net CC_OUT_0: no longer CC2-EXT1.GDO0
- net GND: no longer CC2-EXT1.GND@0, CC2-EXT1.GND@1, IC2.GND, IC2.GND@1, IC2.GND@2, X2.GND1, X2.GND2, X2.GND3, X2.GND4
- net MISO1: no longer CC2-EXT1.MISO
- net MISO2: no longer IC2.MISO
- net MOSI1: no longer CC2-EXT1.MOSI
- net N$3: now also ANT2.TP; no longer X2.ANT
- net RST: no longer IC2.MOSI
- net SCK1: no longer CC2-EXT1.SCLK
- net SCK2: no longer IC2.SCLK
- net VCC: no longer CC2-EXT1.VCC@0, CC2-EXT1.VCC@1, IC2.V+, IC2.V+@1
- net WIZ_CS: no longer IC2.!SCS!
- net WIZ_RST: no longer IC2.RES
Changed lines of the file:
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@@
 <setting verticaltext="up"/>
 </settings>
-<grid distance="50" unitdist="mil" unit="mil" style="lines" multiple="1" display="no" altdistance="0.01" altunitdist="inch" altunit="inch"/>
+<grid distance="0.1" unitdist="inch" unit="inch" style="lines" multiple="1" display="no" altdistance="0.01" altunitdist="inch" altunit="inch"/>
 <layers>
 <layer number="1" name="Top" color="4" fill="1" visible="no" active="no"/>
@@
 <part name="X5" library="adafruit" deviceset="SMACONNECTOR" device="_EDGE_UFL"/>
 <part name="X1" library="adafruit" deviceset="SMACONNECTOR" device="_EDGE_UFL"/>
-<part name="X2" library="adafruit" deviceset="SMACONNECTOR" device="_EDGE_UFL"/>
-<part name="CC2-EXT1" library="wireless" deviceset="CC1101_MODULE3_DIL" device=""/>
-<part name="IC2" library="Martin-Communication" deviceset="LAN-USR-ES1" device=""/>
 <part name="SUPPLY12" library="supply2" deviceset="VCC" device=""/>
 <part name="GND15" library="supply1" deviceset="GND" device=""/>
 <part name="ANT3" library="testpad" deviceset="TP" device="PAD1-13"/>
+<part name="ANT2" library="testpad" deviceset="TP" device="PAD1-13"/>
 </parts>
 <sheets>
@@
 <instance part="X5" gate="G$1" x="63.5" y="228.6"/>
 <instance part="X1" gate="G$1" x="138.43" y="228.6"/>
-<instance part="X2" gate="G$1" x="212.09" y="228.6"/>
-<instance part="CC2-EXT1" gate="G$1" x="38.1" y="177.8"/>
-<instance part="IC2" gate="G$1" x="210.82" y="116.84"/>
 <instance part="SUPPLY12" gate="G$1" x="60.96" y="139.7"/>
 <instance part="GND15" gate="1" x="54.61" y="133.35" rot="R270"/>
 <instance part="ANT3" gate="G$1" x="283.21" y="224.79" rot="R270"/>
+<instance part="ANT2" gate="G$1" x="209.55" y="228.6" rot="R270"/>
 </instances>
 <busses>
@@
 <pinref part="GND11" gate="1" pin="GND"/>
 <wire x1="198.12" y1="222.25" x2="198.12" y2="226.06" width="0.1524" layer="91"/>
-<pinref part="X2" gate="G$1" pin="GND4"/>
-<pinref part="X2" gate="G$1" pin="GND3"/>
-<wire x1="214.63" y1="220.98" x2="209.55" y2="220.98" width="0.1524" layer="91"/>
-<wire x1="209.55" y1="220.98" x2="201.93" y2="220.98" width="0.1524" layer="91"/>
-<wire x1="201.93" y1="220.98" x2="201.93" y2="226.06" width="0.1524" layer="91"/>
-<pinref part="X2" gate="G$1" pin="GND1"/>
 <wire x1="201.93" y1="226.06" x2="201.93" y2="231.14" width="0.1524" layer="91"/>
-<wire x1="201.93" y1="231.14" x2="201.93" y2="236.22" width="0.1524" layer="91"/>
-<wire x1="201.93" y1="236.22" x2="209.55" y2="236.22" width="0.1524" layer="91"/>
-<pinref part="X2" gate="G$1" pin="GND2"/>
-<wire x1="209.55" y1="236.22" x2="214.63" y2="236.22" width="0.1524" layer="91"/>
 <pinref part="CC2" gate="G$1" pin="GND@2"/>
 <wire x1="201.93" y1="231.14" x2="198.12" y2="231.14" width="0.1524" layer="91"/>
 <wire x1="198.12" y1="226.06" x2="201.93" y2="226.06" width="0.1524" layer="91"/>
-<junction x="201.93" y="231.14"/>
-<junction x="201.93" y="226.06"/>
 <junction x="198.12" y="226.06"/>
-<junction x="209.55" y="220.98"/>
-<junction x="209.55" y="236.22"/>
 </segment>
 <segment>
@@
 </segment>
 <segment>
-<pinref part="CC2-EXT1" gate="G$1" pin="GND@0"/>
 <wire x1="38.1" y1="182.88" x2="20.32" y2="182.88" width="0.1524" layer="91"/>
 <label x="22.86" y="182.88" size="1.778" layer="95"/>
 </segment>
 <segment>
-<pinref part="CC2-EXT1" gate="G$1" pin="GND@1"/>
 <wire x1="38.1" y1="180.34" x2="20.32" y2="180.34" width="0.1524" layer="91"/>
 <label x="22.86" y="180.34" size="1.778" layer="95"/>
 </segment>
 <segment>
-<pinref part="IC2" gate="G$1" pin="GND"/>
 <wire x1="198.12" y1="104.14" x2="196.85" y2="104.14" width="0.1524" layer="91"/>
 <wire x1="196.85" y1="104.14" x2="196.85" y2="101.6" width="0.1524" layer="91"/>
-<pinref part="IC2" gate="G$1" pin="GND@1"/>
 <wire x1="196.85" y1="101.6" x2="198.12" y2="101.6" width="0.1524" layer="91"/>
 <wire x1="198.12" y1="101.6" x2="196.85" y2="101.6" width="0.1524" layer="91"/>
 <wire x1="196.85" y1="101.6" x2="196.85" y2="99.06" width="0.1524" layer="91"/>
-<pinref part="IC2" gate="G$1" pin="GND@2"/>
 <wire x1="196.85" y1="99.06" x2="198.12" y2="99.06" width="0.1524" layer="91"/>
 <wire x1="196.85" y1="101.6" x2="189.23" y2="101.6" width="0.1524" layer="91"/>
@@
 </segment>
 <segment>
-<pinref part="IC2" gate="G$1" pin="!SCS!"/>
 <wire x1="198.12" y1="124.46" x2="189.23" y2="124.46" width="0.1524" layer="91"/>
 <label x="190.5" y="124.46" size="1.778" layer="95"/>
@@
 </segment>
 <segment>
-<pinref part="IC2" gate="G$1" pin="MOSI"/>
 <wire x1="198.12" y1="116.84" x2="189.23" y2="116.84" width="0.1524" layer="91"/>
 <label x="190.5" y="116.84" size="1.778" layer="95"/>
@@
 </segment>
 <segment>
-<pinref part="IC2" gate="G$1" pin="RES"/>
 <wire x1="198.12" y1="119.38" x2="189.23" y2="119.38" width="0.1524" layer="91"/>
 <label x="190.5" y="119.38" size="1.778" layer="95"/>
@@
 </segment>
 <segment>
-<pinref part="IC2" gate="G$1" pin="SCLK"/>
 <wire x1="198.12" y1="111.76" x2="189.23" y2="111.76" width="0.1524" layer="91"/>
 <label x="190.5" y="111.76" size="1.778" layer="95"/>
@@
 </segment>
 <segment>
-<pinref part="IC2" gate="G$1" pin="MISO"/>
 <wire x1="198.12" y1="114.3" x2="189.23" y2="114.3" width="0.1524" layer="91"/>
 <label x="190.5" y="114.3" size="1.778" layer="95"/>
@@
 </segment>
 <segment>
-<pinref part="CC2-EXT1" gate="G$1" pin="GDO0"/>
 <wire x1="38.1" y1="187.96" x2="20.32" y2="187.96" width="0.1524" layer="91"/>
 <label x="22.86" y="187.96" size="1.778" layer="95"/>
@@
 </segment>
 <segment>
-<pinref part="CC2-EXT1" gate="G$1" pin="GDO2"/>
 <wire x1="38.1" y1="190.5" x2="20.32" y2="190.5" width="0.1524" layer="91"/>
 <label x="22.86" y="190.5" size="1.778" layer="95"/>
@@
 </segment>
 <segment>
-<pinref part="CC2-EXT1" gate="G$1" pin="VCC@0"/>
 <wire x1="38.1" y1="203.2" x2="20.32" y2="203.2" width="0.1524" layer="91"/>
 <label x="22.86" y="203.2" size="1.778" layer="95"/>
 </segment>
 <segment>
-<pinref part="CC2-EXT1" gate="G$1" pin="VCC@1"/>
 <wire x1="38.1" y1="200.66" x2="20.32" y2="200.66" width="0.1524" layer="91"/>
 <label x="22.86" y="200.66" size="1.778" layer="95"/>
 </segment>
 <segment>
-<pinref part="IC2" gate="G$1" pin="V+"/>
 <wire x1="198.12" y1="132.08" x2="196.85" y2="132.08" width="0.1524" layer="91"/>
 <wire x1="196.85" y1="132.08" x2="196.85" y2="129.54" width="0.1524" layer="91"/>
-<pinref part="IC2" gate="G$1" pin="V+@1"/>
 <wire x1="196.85" y1="129.54" x2="198.12" y2="129.54" width="0.1524" layer="91"/>
 <wire x1="196.85" y1="129.54" x2="189.23" y2="129.54" width="0.1524" layer="91"/>
@@
 </segment>
 <segment>
-<pinref part="CC2-EXT1" gate="G$1" pin="CSN"/>
 <wire x1="38.1" y1="185.42" x2="20.32" y2="185.42" width="0.1524" layer="91"/>
 <label x="22.86" y="185.42" size="1.778" layer="95"/>
@@
 </segment>
 <segment>
-<pinref part="CC2-EXT1" gate="G$1" pin="SCLK"/>
 <wire x1="38.1" y1="195.58" x2="20.32" y2="195.58" width="0.1524" layer="91"/>
 <label x="22.86" y="195.58" size="1.778" layer="95"/>
@@
 </segment>
 <segment>
-<pinref part="CC2-EXT1" gate="G$1" pin="MISO"/>
 <wire x1="38.1" y1="193.04" x2="20.32" y2="193.04" width="0.1524" layer="91"/>
 <label x="22.86" y="193.04" size="1.778" layer="95"/>
@@
 </segment>
 <segment>
-<pinref part="CC2-EXT1" gate="G$1" pin="MOSI"/>
 <wire x1="38.1" y1="198.12" x2="20.32" y2="198.12" width="0.1524" layer="91"/>
 <label x="22.86" y="198.12" size="1.778" layer="95"/>
@@
 <net name="N$3" class="0">
 <segment>
-<pinref part="X2" gate="G$1" pin="ANT"/>
 <pinref part="CC2" gate="G$1" pin="ANT"/>
 <wire x1="204.47" y1="228.6" x2="198.12" y2="228.6" width="0.1524" layer="91"/>
+<pinref part="ANT2" gate="G$1" pin="TP"/>
+<wire x1="204.47" y1="228.6" x2="207.01" y2="228.6" width="0.1524" layer="91"/>
 </segment>
 </net>
 <net name="N$33" class="0">
 <segment>
-<pinref part="IC2" gate="G$1" pin="!INT!"/>
 <wire x1="198.12" y1="106.68" x2="189.23" y2="106.68" width="0.1524" layer="91"/>
 <label x="190.5" y="106.68" size="1.778" layer="95"/>
