File: HW-MAPLE-Large/mapleCUx_large_050.brd (EAGLE design)
At the start: 100 x 59 mm, 37 parts, among them IC31 ATMEGA168-TQFP, X1 SMA, X2 SMA, X3 SMA, X31 M03X2, X4 SMA

Commit message: v50 1Wire -draft
Parts:
- added 1WIRE: (no value), con-lstb:MA03-1
- added 3V3, 5V: (no value), jumper:SJ
- added F1: 1812L, ptc-littlefuse:1812L
- added HMMOD-UART: HM-MOD-UARTDIL, wireless:HM-MOD-UART-DIL
- added IC1: DS2482-100S, 1wire:SO08
- added Q1: BSS84, transistor-small-signal:SOT23
- added R1: 4k7, rcl:R0805
- added R2: 4K7, rcl:R0805
- added R3, R4: 100, rcl:R0805
- added X5: (no value), adafruit:SMA_EDGELAUNCH_UFL
- added ZD1: DS9503P, 1wire:TSOC6
- X1, X2, X3: value SMA -> (none); device sma:SMA -> adafruit:SMA_EDGELAUNCH_UFL
- X4: value SMA -> 1751248; device sma:SMA -> con-phoenix-350:1751248
- moved X4 161.7 mm to (-20.8, -60.2), turned to 0 degrees
- moved X3 99.7 mm to (99.7, 47.6), turned to 180 degrees
- moved X2 36.2 mm to (0.00, 48.3)
- moved LED32 16.1 mm to (97.8, 26.1), turned to 270 degrees
- moved X1 0.63 mm to (99.7, 11.4)
- renumbered X31 to ARDU_PRG
Connections:
- new net N$34: IC1.2, R3.1
- new net N$43: IC1.4, R2.2
- new net N$44: IC1.5, R1.2
- new net N$45: F1.P$2, X4.1
- new net N$47: IC1.6, Q1.1
- new net N$48: Q1.3, R3.2, ZD1.1
- new net N$50: 1WIRE.2, ZD1.6
- new net N$51: 1WIRE.3, ZD1.5
- new net N$52: Q1.2, R4.1
- new net VDD: 1WIRE.1, 3V3.2, 5V.1, F1.P$1, IC1.1, R1.1, R2.1, R4.2
- net +5V: now also 5V.2
- net GND: now also HMMOD-UART.2, IC1.3, IC1.7, IC1.8, X4.2, X5.GND@1, X5.GND@2, X5.GND@3, X5.GND@4, ZD1.2; no longer X4.GND@1, X4.GND@2, X4.GND@3, X4.GND@4
- net N$1: now also CC1.ANT, X1.P; no longer CC2.ANT, X3.1
- net N$2: now also X3.P; no longer X4.1
- net N$3: now also CC2.ANT, X2.P; no longer CC1.ANT, X1.1
- net N$4: now also X5.P; no longer X2.1
- net RX1: now also HMMOD-UART.5
- net TX1: now also HMMOD-UART.6
- net VCC: now also 3V3.1, HMMOD-UART.1
Routing:
- net VCC: track 270.7 -> 0.00 mm, vias 2 -> 0
- net MISO1: track 157.7 -> 0.00 mm, vias 2 -> 0
- net MOSI1: track 156.7 -> 0.00 mm, vias 1 -> 0
- net SCK1: track 148.0 -> 0.00 mm
- net TX-MAPLE: track 114.0 -> 0.00 mm, vias 2 -> 0
- net RX-MAPLE: track 102.0 -> 0.00 mm, vias 2 -> 0
- net CC_CS1: track 97.9 -> 0.00 mm, vias 2 -> 0
- net RST: track 87.2 -> 0.00 mm
- net CC_OUT_1: track 84.0 -> 0.00 mm
- net CC_IN_1: track 83.9 -> 0.00 mm
- net CC_IN_3: track 72.8 -> 0.00 mm
- net CE-A: track 70.2 -> 0.00 mm
- net MOSI-A: track 67.0 -> 0.00 mm
- net SCK2: track 66.8 -> 0.00 mm
- net CSN-A: track 63.8 -> 0.00 mm
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Other:
- outline, holes or cut-outs redrawn
- board text added: "MAPLE CUN Lage Version A 1.3"
- board text added: "MAPLE CUN Large Version A 1.3"
- board text removed: "MAPLE CUN Lage Version A 1.2"
