File: HW-MAPLE-Large/mapleCUx_large_052.brd (EAGLE design)
At the start: 100 x 59 mm, 50 parts, among them IC1 DS2482-100S, IC31 ATMEGA168-TQFP, Q1 BSS84, X4 1751248

Commit message: v52 1Wire v2
Parts:
- removed R3: 100, rcl:R0805
- removed W5500NIREN: (no value), con-lstb:MA05-2
- moved F1 136.7 mm to (89.9, 10.7), flipped to the bottom, turned to 270 degrees
- moved X4 124.6 mm to (87.1, 2.03)
- moved ZD1 124.2 mm to (89.7, 17.3), flipped to the bottom
- moved 5V 113.9 mm to (73.7, 8.89), flipped to the bottom
- moved 3V3 113.7 mm to (73.7, 12.7), flipped to the bottom, turned to 180 degrees
- moved R4 111.1 mm to (85.1, 10.2), flipped to the bottom
- moved Q1 109.4 mm to (89.9, 5.59), flipped to the bottom, turned to 90 degrees
- moved R2 98.0 mm to (80.0, 7.62), flipped to the bottom, turned to 180 degrees
- moved R1 97.5 mm to (80.0, 10.2), flipped to the bottom, turned to 180 degrees
- moved IC1 96.2 mm to (81.5, 15.2), flipped to the bottom, turned to 90 degrees
- moved 1WIRE 93.2 mm to (78.5, 1.78)
Connections:
- removed net N$34: IC1.2, R3.1
- removed net N$43: IC1.4, R2.2
- removed net N$44: IC1.5, R1.2
- removed net N$50: 1WIRE.2, ZD1.6
- new net N$21: 1WIRE.2, ZD1.1
- net +5V: no longer W5500NIREN.1
- net CC_CS2: now also IC1.5, R1.2
- net CC_IN_2: now also IC1.4, R2.2
- net GND: now also ZD1.5; no longer W5500NIREN.3, ZD1.2
- net MISO2: no longer W5500NIREN.4
- net N$48: now also IC1.2, ZD1.6; no longer R3.2, ZD1.1
- net N$51: now also ZD1.2; no longer ZD1.5
- net RST: no longer W5500NIREN.6
- net SCK2: no longer W5500NIREN.10
- net WIZ_CS: no longer W5500NIREN.8
- net WIZ_RST: no longer W5500NIREN.5
Routing:
- net VCC: track 0.00 -> 287.6 mm, vias 0 -> 1
- net MISO1: track 0.00 -> 169.5 mm, vias 0 -> 1
- net SCK1: track 0.00 -> 157.2 mm, vias 0 -> 1
- net MOSI1: track 0.00 -> 149.7 mm, vias 0 -> 2
- net TX-MAPLE: track 0.00 -> 103.2 mm, vias 0 -> 2
- net RX-MAPLE: track 0.00 -> 90.5 mm, vias 0 -> 2
- net CC_OUT_1: track 0.00 -> 89.6 mm, vias 0 -> 2
- net MISO-A: track 0.00 -> 86.7 mm, vias 0 -> 2
- net TX1: track 0.00 -> 85.7 mm
- net CC_CS1: track 0.00 -> 78.9 mm, vias 0 -> 1
- net CC_IN_3: track 0.00 -> 73.3 mm
- net RX1: track 0.00 -> 72.5 mm, vias 0 -> 1
- net IRQ-A: track 0.00 -> 70.1 mm
- net CSN-A: track 0.00 -> 67.0 mm, vias 0 -> 1
- net CC_IN_1: track 0.00 -> 65.9 mm
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