File: HW-MAPLE-Large/mapleCUx_large_052.sch (EAGLE design)
At the start: 50 parts, among them IC1 DS2482-100S, IC31 ATMEGA168-TQFP, Q1 BSS84, X4 1751248

Commit message: v52 1Wire v2
Parts:
- removed R3: 100, rcl:R-EU_R0805
- removed W5500NIREN: (no value), con-lstb:MA05-2
Connections:
- removed net N$34: IC1G$1.1W, R3.1
- removed net N$43: IC1G$1.SCL, R2.2
- removed net N$44: IC1G$1.SDA, R1.2
- removed net N$50: 1WIRE.2, ZD1.P$4
- new net N$21: 1WIRE.2, ZD1.P$1
- net +5V: no longer W5500NIREN.1
- net CC_CS2: now also IC1G$1.SDA, R1.2
- net CC_IN_2: now also IC1G$1.SCL, R2.2
- net GND: now also ZD1.P$3; no longer W5500NIREN.3, ZD1.P$2
- net MISO2: no longer W5500NIREN.4
- net N$48: now also IC1G$1.1W, ZD1.P$4; no longer R3.2, ZD1.P$1
- net N$51: now also ZD1.P$2; no longer ZD1.P$3
- net RST: no longer W5500NIREN.6
- net SCK2: no longer W5500NIREN.10
- net WIZ_CS: no longer W5500NIREN.8
- net WIZ_RST: no longer W5500NIREN.5
Other:
- note added: "Funktioniert nur ohne Transceiver CC2 !"
- moved on the sheet: 1WIRE, 3V3, 5V, F1, IC1, Q1, R1, R2, R4, X4-1, X4-2, ZD1
