File: HW-MAPLE-Large/mapleCUx_large_056.brd (EAGLE design)
At the start: 100 x 59 mm, 48 parts, among them IC1 DS2482-100S, IC31 ATMEGA168-TQFP, Q1 BSS84, X4 1751248

Commit message: Large 056
Parts:
- removed U$3: USR-ES1, Martin:USR-ES1
- added C10: 100uF, rcl:E5-8,5
- added C8: 220p, rcl:C0805
- added C9: 22p, rcl:C0805
- added GND: (no value), jumper:SJ
- added IC2: LAN-USR-ES1, Martin-Communication:USR-ES1
- added R3, R5: 60, rcl:R0805
- added RS485: MAX487ECSA+, Maxim_By_element14_Batch_1:SOIC127P600X175-8N
- 1WIRE: device con-lstb:MA03-1 -> con-lstb:MA04-1
- C5: device rcl:C1210 -> rcl:R/2012-12W
- moved CTX-DB 46.6 mm to (8.58, 28.4), flipped to the bottom, turned to 90 degrees
- moved R32 14.2 mm to (94.6, 30.2), turned to 270 degrees
- moved ZD1 12.8 mm to (80.8, 8.13), turned to 90 degrees
- moved R1 12.6 mm to (88.9, 19.1), turned to 0 degrees
- moved R2 10.9 mm to (83.8, 17.8), turned to 270 degrees
- moved Q1 8.54 mm to (85.6, 13.0), turned to 180 degrees
- moved R4 7.41 mm to (88.9, 16.5), turned to 180 degrees
- moved X4 6.48 mm to (93.5, 3.30)
- moved 1WIRE 4.58 mm to (82.8, 3.30), turned to 180 degrees
- moved C4 3.17 mm to (72.4, 54.2)
- moved C32 1.84 mm to (80.0, 29.2)
- moved R34 1.61 mm to (77.5, 29.2), flipped to the top, turned to 270 degrees
- moved IC1 1.55 mm to (80.0, 15.5), turned to 0 degrees
- moved UART1 1.42 mm to (41.9, 12.1)
- moved UART0 1.42 mm to (38.0, 12.1)
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Connections:
- removed net N$46: U$3.NINT
- removed net N$49: U$3.PWDN
- removed net N$51: 1WIRE.3, ZD1.2
- new net 1W: 1WIRE.2, R5.2, RS485.6, ZD1.1
- new net 2W: 1WIRE.3, R3.2, RS485.7
- new net GD: 1WIRE.4, GND.2, ZD1.2
- new net N$33: IC2.6
- new net RO-A: RS485.1, U$2.D8
- net CE-A: now also RS485.4
- net GND: now also C10.-, C5.-, C8.2, C9.1, GND.1, IC2.1, IC2.12, IC2.2, RS485.5; no longer C5.2, U$3.GND, U$3.GND2, U$3.GND3
- net IRQ-A: now also RS485.2, RS485.3
- net MISO2: now also IC2.7; no longer U$3.MISO
- net N$21: now also C8.1, R3.1, R5.1; no longer 1WIRE.2, ZD1.1
- net RST: now also IC2.3; no longer U$3.MOSI
- net SCK2: now also IC2.4, IC2.5; no longer U$3.SCLK
- net VCC: now also C10.+, C5.+, IC2.10, IC2.11; no longer C5.1, U$3.VIN3.3, U$3.VIN3.3B
- net VDD: now also C9.2, RS485.8
- net WIZ_CS: no longer U$3.NSS
- net WIZ_RST: now also IC2.8; no longer U$3.NRESET
Routing:
- net 1W: track 0.00 -> 149.8 mm, vias 0 -> 2
- net RO-A: track 0.00 -> 124.5 mm, vias 0 -> 1
- net CC_CS2: track 52.8 -> 163.5 mm, vias 0 -> 2
- net VDD: track 32.2 -> 127.6 mm, vias 0 -> 2
- net 2W: track 0.00 -> 95.4 mm, vias 0 -> 1
- net CC_IN_2: track 44.1 -> 125.5 mm, vias 0 -> 2
- net CE-A: track 43.2 -> 112.8 mm, vias 1 -> 2
- net SWO/TDO: track 58.8 -> 14.3 mm, vias 1 -> 0
- net NRESET: track 51.9 -> 7.70 mm, vias 2 -> 0
- net WIZ_CS: track 53.9 -> 19.4 mm
- net IRQ-A: track 70.1 -> 103.3 mm, vias 0 -> 2
- net N$51: track 27.8 -> 0.00 mm
- net MISO-A: track 86.7 -> 60.1 mm, vias 2 -> 1
- net SWCLK/TCK: track 34.5 -> 15.0 mm
- net MOSI1: track 149.7 -> 168.6 mm, vias 2 -> 0
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