File: HW-MAPLE-Large/mapleCUx_large_056.sch (EAGLE design)
At the start: 48 parts, among them IC1 DS2482-100S, IC31 ATMEGA168-TQFP, Q1 BSS84, X4 1751248

Commit message: Large 056
Parts:
- removed U$3: USR-ES1, Martin:USR-ES1
- added C10: 100uF, rcl:CPOL-EUE5-8.5
- added C8: 220p, rcl:C-EUC0805
- added C9: 22p, rcl:C-EUC0805
- added GND: (no value), jumper:SJ
- added IC2: LAN-USR-ES1, Martin-Communication:LAN-USR-ES1
- added R3, R5: 60, rcl:R-EU_R0805
- added RS485: MAX487ECSA+, Maxim_By_element14_Batch_1:MAX487ECSA+
- 1WIRE: device con-lstb:MA03-1 -> con-lstb:MA04-1
- C5: device rcl:C-EUC1210 -> rcl:CPOL-EUR/2012-12W
Connections:
- removed net N$46: U$3.6
- removed net N$49: U$3.10
- removed net N$51: 1WIRE.3, ZD1.P$2
- new net 1W: 1WIRE.2, R5.2, RS485.A, ZD1.P$1
- new net 2W: 1WIRE.3, R3.2, RS485.B
- new net GD: 1WIRE.4, GND.2, ZD1.P$2
- new net N$33: IC2.!INT!
- new net RO-A: RS485.RO, U$2.D8
- net CE-A: now also RS485.DI
- net GND: now also C10.-, C5.-, C8.2, C9.1, GND.1, IC2.GND, IC2.GND@1, IC2.GND@2, RS485.GND; no longer C5.2, U$3.1, U$3.2, U$3.7
- net IRQ-A: now also RS485.DE, RS485.~RE
- net MISO2: now also IC2.MISO; no longer U$3.12
- net N$21: now also C8.1, R3.1, R5.1; no longer 1WIRE.2, ZD1.P$1
- net RST: now also IC2.MOSI; no longer U$3.3
- net SCK2: now also IC2.!SCS!, IC2.SCLK; no longer U$3.4
- net VCC: now also C10.+, C5.+, IC2.V+, IC2.V+@1; no longer C5.1, U$3.8, U$3.9
- net VDD: now also C9.2, RS485.VCC
- net WIZ_CS: no longer U$3.5
- net WIZ_RST: now also IC2.RES; no longer U$3.11
Other:
- note added: "ARM-Debugger"
- note added: "Alternativ:"
- note added: "Alternative Minimal-Version:"
- note added: "HomeMatic"
- note added: "Optional !"
- note added: "Selbe Leiste als 1Wire..."
- note added: "VDD-Config siehe 1Wire..."
- note removed: "Homematic"
- moved on the sheet: ARDU_PRG, C31, C32, C7, HMMOD-UART, IC31, LED32, NRF24L01+, R32, R34, W5100, X1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
