File: HW-MAPLE-Large/mapleCUx_large_082.sch (EAGLE design)
At the start: 54 parts, among them IC1 DS2482-100S, IC2 LAN-USR-ES1, Q1 BSS84, X4 1751248, X7 1751264

Commit message: Large 082 Maple moved to Top...
Parts:
- added C12: 22pF, rcl:C-EUC0805
- added U$3: ESP01, esp8266modules:ESP01
- IC1: value DS2482-100S -> DS2482
- renumbered CC_X4 to CC_X3
Connections:
- net GND: now also C12.2, U$3.GND
- net N$11: now also U$3.GPIO0
- net N$17: now also U$3.CH_PD
- net RX_DBG: now also U$3.TXD
- net SCK2: no longer IC2.!SCS!
- net TX_DBG: now also U$3.RXD
- net VCC: now also C12.1, U$3.VCC
- net WIZ_CS: now also IC2.!SCS!
Other:
- note removed: "Alternativ:"
- note removed: "W5500 NiRen 55x28mm Drill dist 23,1mm"
