File: HW-MAPLE-Large/mapleCUx_large_084.brd (EAGLE design)
At the start: 100 x 59 mm, 56 parts, among them IC1 DS2482, IC2 LAN-USR-ES1, Q1 BSS84, X4 1751248, X7 1751264

Commit message: Cleanup + Stripped Version
Changed lines of the file:
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@@
 <signal name="N$37">
 <via x="16.51" y="55.88" extent="1-16" drill="0.304796875" diameter="0.6096"/>
+<via x="14.986" y="53.34" extent="1-16" drill="0.304796875" diameter="0.6096"/>
+<via x="21.59" y="55.88" extent="1-16" drill="0.304796875" diameter="0.6096"/>
+<via x="18.796" y="53.34" extent="1-16" drill="0.304796875" diameter="0.6096"/>
+<via x="79.502" y="56.896" extent="1-16" drill="0.304796875" diameter="0.6096"/>
+<via x="87.376" y="49.53" extent="1-16" drill="0.304796875" diameter="0.6096"/>
+<via x="82.804" y="56.896" extent="1-16" drill="0.304796875" diameter="0.6096"/>
+<via x="16.002" y="49.276" extent="1-16" drill="0.304796875" diameter="0.6096"/>
+<via x="86.106" y="56.896" extent="1-16" drill="0.304796875" diameter="0.6096"/>
+<via x="10.414" y="43.434" extent="1-16" drill="0.304796875" diameter="0.6096"/>
+<via x="88.9" y="56.896" extent="1-16" drill="0.304796875" diameter="0.6096"/>
+<via x="84.582" y="46.99" extent="1-16" drill="0.304796875" diameter="0.6096"/>
+<via x="91.948" y="56.896" extent="1-16" drill="0.304796875" diameter="0.6096"/>
+<via x="69.85" y="1.524" extent="1-16" drill="0.304796875" diameter="0.6096"/>
+<via x="21.082" y="2.794" extent="1-16" drill="0.304796875" diameter="0.6096"/>
+<via x="17.272" y="3.048" extent="1-16" drill="0.304796875" diameter="0.6096"/>
+<via x="13.97" y="3.048" extent="1-16" drill="0.304796875" diameter="0.6096"/>
+<via x="11.938" y="28.194" extent="1-16" drill="0.304796875" diameter="0.6096"/>
+<via x="55.372" y="33.528" extent="1-16" drill="0.304796875" diameter="0.6096"/>
+<via x="13.208" y="46.736" extent="1-16" drill="0.304796875" diameter="0.6096"/>
+<via x="88.646" y="43.18" extent="1-16" drill="0.304796875" diameter="0.6096"/>
+<via x="81.534" y="41.91" extent="1-16" drill="0.304796875" diameter="0.6096"/>
+<via x="74.676" y="33.274" extent="1-16" drill="0.304796875" diameter="0.6096"/>
+<via x="59.436" y="20.066" extent="1-16" drill="0.304796875" diameter="0.6096"/>
+<via x="51.308" y="15.24" extent="1-16" drill="0.304796875" diameter="0.6096"/>
+<via x="86.868" y="8.89" extent="1-16" drill="0.304796875" diameter="0.6096"/>
 </signal>
 <signal name="N$38">
@@
 </signal>
 <signal name="N$39">
-<via x="93.98" y="41.91" extent="1-16" drill="0.304796875" diameter="0.6096"/>
+<via x="88.138" y="46.736" extent="1-16" drill="0.304796875" diameter="0.6096"/>
 </signal>
 <signal name="N$4">
@@
 </signal>
 <signal name="N$23">
-<via x="13.335" y="39.37" extent="1-16" drill="0.3048" diameter="0.6096"/>
+<via x="13.589" y="44.196" extent="1-16" drill="0.3048" diameter="0.6096"/>
 </signal>
 <signal name="N$25">
 <via x="17.145" y="39.37" extent="1-16" drill="0.3048" diameter="0.6096"/>
 </signal>
-<signal name="N$31">
-<via x="71.755" y="57.15" extent="1-16" drill="0.3048" diameter="0.6096"/>
-</signal>
 <signal name="N$35">
