File: Adapter-for-Stamps/Adapter-Stamps-005.brd (EAGLE design)
At the start: 36.5 x 18.1 mm, 5 parts, among them X2 SMA

Commit message: V2 Large, Small-Update
Parts:
- removed X2: SMA, sma:SMA
- added X1: (no value), adafruit:SMA_EDGELAUNCH_UFL
Connections:
- new net N$1: CC0.ANT, X1.P
- new net N$3: CC0.GND@1, CC0.GND@2, X1.GND@1, X1.GND@2, X1.GND@3, X1.GND@4
- net ANT: no longer CC0.ANT, X2.1
- net GND: no longer CC0.GND@1, CC0.GND@2, X2.GND@1, X2.GND@2, X2.GND@3, X2.GND@4
Routing:
- net GND: track 113.4 -> 89.4 mm, vias 27 -> 25
- net N$3: track 0.00 -> 22.8 mm, vias 0 -> 1
- net ANT: track 5.10 -> 1.29 mm
- net N$1: track 0.00 -> 3.09 mm
Other:
- board text added: "Stamp-Adapter V2 (Mini-)Stamp, SMA, U.FL"
- board text added: "www.neuby.de"
Changed lines of the file:
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@@
 <text x="34.925" y="8.89" size="0.8128" layer="25">SO</text>
 <text x="34.925" y="6.35" size="0.8128" layer="25">SI</text>
+<text x="9.144" y="5.461" size="0.6096" layer="25" font="vector">Stamp-Adapter V2
+(Mini-)Stamp, SMA, U.FL</text>
+<text x="19.812" y="5.207" size="0.6096" layer="26" font="vector" rot="MR0">Stamp-Adapter V2
+(Mini-)Stamp, SMA, U.FL</text>
+<text x="19.558" y="15.494" size="0.6096" layer="26" font="vector" rot="MR0">www.neuby.de</text>
 </plain>
 <attributes>
@@
 <elements>
 <element name="CC0" library="wireless" package="CC1101_MODULE1_SMD" value="CC1101_MODULE1SMD" x="26.035" y="16.51" rot="R180"/>
-<element name="X2" library="sma" package="SMA" value="SMA" x="1.27" y="10.16"/>
 <element name="CC_X0" library="con-lstb" package="MA05-2" value="" x="32.385" y="9.525" smashed="yes" rot="R90">
 <attribute name="OC_NEWARK" value="unknown" x="32.385" y="9.525" size="1.778" layer="27" rot="R90" display="off"/>
@@
 </element>
 <element name="C1" library="rcl" package="C0805" value="22pF" x="28.575" y="3.81" smashed="yes" rot="R270"/>
-<element name="RADIO0B" library="Martin-Communication" package="CC1101_MODULE1_SMD" value="CC1101_MODULE1SMALL" x="23.2156" y="14.9352" rot="R180"/>
+<element name="RADIO0B" library="Martin-Communication" package="CC1101_MODULE1_SMD" value="CC1101_MODULE1SMALL" x="23.2156" y="14.9352" smashed="yes" rot="R180"/>
+<element name="X1" library="adafruit" package="SMA_EDGELAUNCH_UFL" value="" x="1.016" y="10.668"/>
 </elements>
 <signals>
 <signal name="GND">
 <contactref element="CC0" pad="GND@0"/>
-<contactref element="CC0" pad="GND@1"/>
-<contactref element="CC0" pad="GND@2"/>
-<contactref element="X2" pad="GND@1"/>
-<contactref element="X2" pad="GND@3"/>
-<contactref element="X2" pad="GND@2"/>
-<contactref element="X2" pad="GND@4"/>
 <contactref element="CC_X0" pad="9"/>
 <contactref element="CC_X0" pad="10"/>
@@
 <contactref element="RADIO0B" pad="GND@1"/>
 <contactref element="RADIO0B" pad="GND@2"/>
-<via x="1.905" y="16.51" extent="1-16" drill="0.6" shape="square"/>
-<via x="3.81" y="16.51" extent="1-16" drill="0.6" shape="square"/>
 <via x="1.905" y="2.54" extent="1-16" drill="0.6" shape="square"/>
 <via x="3.81" y="2.54" extent="1-16" drill="0.6" shape="square"/>
@@
 <wire x1="7.8232" y1="8.1026" x2="7.2644" y2="8.1026" width="0.4064" layer="1"/>
 <wire x1="8.1026" y1="8.382" x2="7.8232" y2="8.1026" width="0.4064" layer="1"/>
-<wire x1="7.2644" y1="8.1026" x2="7.035" y2="8.01" width="0.4064" layer="1"/>
 <wire x1="8.1026" y1="8.382" x2="8.3266" y2="8.5542" width="0.4064" layer="1"/>
 <wire x1="3.6322" y1="2.5146" x2="1.9558" y2="2.5146" width="0.4064" layer="1"/>
@@
 <wire x1="3.6322" y1="7.2644" x2="3.6322" y2="2.794" width="0.4064" layer="1"/>
 <wire x1="3.6322" y1="2.794" x2="3.81" y2="2.54" width="0.4064" layer="1"/>
-<wire x1="3.6322" y1="7.2644" x2="3.3854" y2="7.4274" width="0.4064" layer="1"/>
-<wire x1="3.9116" y1="7.8232" x2="6.985" y2="7.8232" width="0.4064" layer="1"/>
-<wire x1="3.6322" y1="7.5438" x2="3.9116" y2="7.8232" width="0.4064" layer="1"/>
-<wire x1="6.985" y1="7.8232" x2="7.035" y2="8.01" width="0.4064" layer="1"/>
-<wire x1="3.6322" y1="7.5438" x2="3.3854" y2="7.4274" width="0.4064" layer="1"/>
 <wire x1="3.6322" y1="2.794" x2="3.6322" y2="7.2644" width="0.4064" layer="16"/>
-<wire x1="3.6322" y1="7.2644" x2="3.3854" y2="7.4274" width="0.4064" layer="16"/>
 <wire x1="3.6322" y1="2.794" x2="3.81" y2="2.54" width="0.4064" layer="16"/>
 <wire x1="34.0868" y1="15.0876" x2="34.0868" y2="17.0434" width="0.4064" layer="1"/>
@@
 <wire x1="7.8232" y1="12.8524" x2="7.2644" y2="12.8524" width="0.4064" layer="1"/>
 <wire x1="8.1026" y1="12.573" x2="7.8232" y2="12.8524" width="0.4064" layer="1"/>
-<wire x1="7.2644" y1="12.8524" x2="7.035" y2="13.09" width="0.4064" layer="1"/>
 <wire x1="8.1026" y1="12.573" x2="8.3266" y2="12.5542" width="0.4064" layer="1"/>
-<wire x1="3.6322" y1="16.4846" x2="1.9558" y2="16.4846" width="0.4064" layer="1"/>
-<wire x1="1.9558" y1="16.4846" x2="1.905" y2="16.51" width="0.4064" layer="1"/>
-<wire x1="3.6322" y1="16.4846" x2="3.81" y2="16.51" width="0.4064" layer="1"/>
-<wire x1="3.6322" y1="13.1318" x2="3.6322" y2="16.4846" width="0.4064" layer="1"/>
-<wire x1="3.6322" y1="16.4846" x2="3.81" y2="16.51" width="0.4064" layer="1"/>
-<wire x1="3.6322" y1="13.1318" x2="3.3854" y2="12.8926" width="0.4064" layer="1"/>
-<wire x1="3.6322" y1="13.1318" x2="6.985" y2="13.1318" width="0.4064" layer="1"/>
-<wire x1="6.985" y1="13.1318" x2="7.035" y2="13.09" width="0.4064" layer="1"/>
-<wire x1="3.6322" y1="13.1318" x2="3.3854" y2="12.8926" width="0.4064" layer="1"/>
 <wire x1="10.6172" y1="15.367" x2="10.6172" y2="17.0434" width="0.4064" layer="1"/>
 <wire x1="8.1026" y1="12.8524" x2="10.6172" y2="15.367" width="0.4064" layer="1"/>
@@
 <wire x1="31.0134" y1="14.8082" x2="31.115" y2="14.605" width="0.4064" layer="16"/>
 <wire x1="20.955" y1="17.0434" x2="20.955" y2="17.145" width="0.4064" layer="16"/>
-<wire x1="3.6322" y1="16.4846" x2="3.6322" y2="13.1318" width="0.4064" layer="16"/>
-<wire x1="3.6322" y1="13.1318" x2="3.3854" y2="12.8926" width="0.4064" layer="16"/>
-<wire x1="3.6322" y1="16.4846" x2="3.81" y2="16.51" width="0.4064" layer="16"/>
-<wire x1="3.3528" y1="12.8524" x2="3.3528" y2="7.5438" width="0.4064" layer="16"/>
-<wire x1="3.3528" y1="7.5438" x2="3.3854" y2="7.4274" width="0.4064" layer="16"/>
-<wire x1="3.3528" y1="12.8524" x2="3.3854" y2="12.8926" width="0.4064" layer="16"/>
 <wire x1="3.9116" y1="2.5146" x2="10.6172" y2="2.5146" width="0.4064" layer="1"/>
 <wire x1="10.6172" y1="2.5146" x2="10.795" y2="2.54" width="0.4064" layer="1"/>
@@
 </signal>
 <signal name="ANT">
-<contactref element="CC0" pad="ANT"/>
-<contactref element="X2" pad="1"/>
 <contactref element="RADIO0B" pad="ANT"/>
 <wire x1="8.3266" y1="10.5542" x2="7.0392" y2="10.5542" width="0.4064" layer="1"/>
-<wire x1="7.0392" y1="10.5542" x2="7.035" y2="10.55" width="0.4064" layer="1"/>
-<wire x1="3.3854" y1="10.16" x2="5.08" y2="10.16" width="1.27" layer="1"/>
-<wire x1="5.08" y1="10.16" x2="5.334" y2="10.414" width="1.27" layer="1"/>
-<wire x1="5.334" y1="10.414" x2="5.588" y2="10.414" width="0.8128" layer="1"/>
-<wire x1="5.588" y1="10.414" x2="5.715" y2="10.541" width="0.8128" layer="1"/>
-<wire x1="5.715" y1="10.541" x2="7.026" y2="10.541" width="0.8128" layer="1"/>
-<wire x1="7.026" y1="10.541" x2="7.035" y2="10.55" width="0.8128" layer="1"/>
+</signal>
+<signal name="N$3">
+<contactref element="X1" pad="GND@4"/>
+<contactref element="X1" pad="GND@3"/>
+<contactref element="X1" pad="GND@2"/>
+<contactref element="X1" pad="GND@1"/>
+<contactref element="CC0" pad="GND@1"/>
+<contactref element="CC0" pad="GND@2"/>
+<wire x1="1.6764" y1="9.4996" x2="1.8161" y2="9.3599" width="0.4064" layer="1"/>
+<wire x1="1.8161" y1="9.3599" x2="2.794" y2="8.382" width="0.4064" layer="1"/>
+<wire x1="1.6764" y1="12.0142" x2="1.6764" y2="9.4996" width="0.4064" layer="1"/>
+<wire x1="2.794" y1="13.1318" x2="2.4511" y2="12.7889" width="0.4064" layer="1"/>
+<wire x1="2.4511" y1="12.7889" x2="1.6764" y2="12.0142" width="0.4064" layer="1"/>
+<wire x1="2.794" y1="8.382" x2="3.048" y2="8.128" width="0.4064" layer="1"/>
+<wire x1="2.794" y1="13.1318" x2="3.048" y2="13.208" width="0.4064" layer="1"/>
+<wire x1="1.9558" y1="8.9408" x2="1.9558" y2="9.4996" width="0.4064" layer="16"/>
+<wire x1="2.794" y1="8.1026" x2="1.9558" y2="8.9408" width="0.4064" layer="16"/>
+<wire x1="1.9558" y1="9.4996" x2="1.8161" y2="9.3599" width="0.4064" layer="1"/>
+<wire x1="2.794" y1="8.1026" x2="3.048" y2="8.128" width="0.4064" layer="16"/>
+<wire x1="3.0734" y1="8.382" x2="3.0734" y2="13.1318" width="0.4064" layer="16"/>
+<wire x1="3.0734" y1="13.1318" x2="3.048" y2="13.208" width="0.4064" layer="16"/>
+<wire x1="3.0734" y1="8.382" x2="3.048" y2="8.128" width="0.4064" layer="16"/>
+<via x="1.9558" y="9.4996" extent="1-16" drill="0.3048"/>
+<wire x1="7.035" y1="13.09" x2="4.064" y2="13.09" width="0.4064" layer="1"/>
+<wire x1="4.064" y1="13.09" x2="4.064" y2="13.208" width="0.4064" layer="1"/>
+<wire x1="4.064" y1="13.208" x2="2.4511" y2="13.208" width="0.4064" layer="1"/>
+<wire x1="2.4511" y1="13.208" x2="2.4511" y2="12.7889" width="0.4064" layer="1"/>
+<wire x1="7.035" y1="8.01" x2="3.048" y2="8.01" width="0.4064" layer="1"/>
+<wire x1="3.048" y1="8.01" x2="3.048" y2="8.128" width="0.4064" layer="1"/>
+</signal>
+<signal name="N$1">
+<contactref element="CC0" pad="ANT"/>
+<contactref element="X1" pad="P"/>
+<wire x1="7.035" y1="10.55" x2="4.064" y2="10.55" width="0.4064" layer="1"/>
+<wire x1="4.064" y1="10.55" x2="4.064" y2="10.668" width="0.4064" layer="1"/>
 </signal>
 </signals>
 </board>
 </drawing>
+<compatibility>
+<note version="6.3" minversion="6.2.2" severity="warning">
+Since Version 6.2.2 text objects can contain more than one line,
+which will not be processed correctly with this version.
+</note>
+</compatibility>
 </eagle>
