File: Adapter-for-Stamps/Adapter-Stamps-005.sch (EAGLE design)
At the start: 5 parts, among them X2 SMA

Commit message: V2 Large, Small-Update
Parts:
- removed X2: SMA, sma:SMA
- added X1: (no value), adafruit:SMACONNECTOR_EDGE_UFL
Connections:
- new net N$1: CC0.ANT, X1.ANT
- new net N$3: CC0.GND@2, CC0.GND@3, X1.GND1, X1.GND2, X1.GND3, X1.GND4
- net ANT: no longer CC0.ANT, X2.1
- net GND: no longer CC0.GND@2, CC0.GND@3, X2.2, X2.3, X2.4, X2.5
Changed lines of the file:
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@@
 <setting verticaltext="up"/>
 </settings>
-<grid distance="0.1" unitdist="inch" unit="inch" style="lines" multiple="1" display="no" altdistance="0.01" altunitdist="inch" altunit="inch"/>
+<grid distance="50" unitdist="mil" unit="mil" style="lines" multiple="1" display="no" altdistance="0.01" altunitdist="inch" altunit="inch"/>
 <layers>
 <layer number="1" name="Top" color="4" fill="1" visible="no" active="no"/>
@@
 <parts>
 <part name="CC0" library="wireless" deviceset="CC1101_MODULE1" device="SMD"/>
-<part name="X2" library="sma" deviceset="SMA" device=""/>
-<part name="GND8" library="supply1" deviceset="GND" device=""/>
 <part name="GND9" library="supply1" deviceset="GND" device=""/>
 <part name="SUPPLY7" library="supply2" deviceset="VCC" device=""/>
@@
 <part name="C1" library="rcl" deviceset="C-EU" device="C0805" value="22pF"/>
 <part name="RADIO0B" library="Martin-Communication" deviceset="CC1101_MODULE1" device="SMALL"/>
+<part name="X1" library="adafruit" deviceset="SMACONNECTOR" device="_EDGE_UFL"/>
 </parts>
 <sheets>
@@
 <instances>
 <instance part="CC0" gate="G$1" x="-35.56" y="123.19"/>
-<instance part="X2" gate="G1" x="-15.24" y="130.81" rot="R180"/>
-<instance part="GND8" gate="1" x="-20.32" y="123.19"/>
 <instance part="GND9" gate="1" x="-72.39" y="138.43" rot="R270"/>
 <instance part="SUPPLY7" gate="G$1" x="-58.42" y="149.86"/>
@@
 <instance part="C1" gate="G$1" x="-66.04" y="144.78" rot="R90"/>
 <instance part="RADIO0B" gate="G$1" x="-35.56" y="165.1"/>
+<instance part="X1" gate="G$1" x="-12.7" y="130.81"/>
 </instances>
 <busses>
@@
 </segment>
 <segment>
-<pinref part="CC0" gate="G$1" pin="GND@2"/>
-<pinref part="X2" gate="G1" pin="2"/>
-<wire x1="-25.4" y1="133.35" x2="-20.32" y2="133.35" width="0.1524" layer="91"/>
-<pinref part="X2" gate="G1" pin="4"/>
-<wire x1="-20.32" y1="133.35" x2="-17.78" y2="133.35" width="0.1524" layer="91"/>
-<wire x1="-17.78" y1="135.89" x2="-20.32" y2="135.89" width="0.1524" layer="91"/>
-<wire x1="-20.32" y1="135.89" x2="-20.32" y2="134.62" width="0.1524" layer="91"/>
-<pinref part="X2" gate="G1" pin="3"/>
-<wire x1="-20.32" y1="134.62" x2="-20.32" y2="133.35" width="0.1524" layer="91"/>
-<wire x1="-17.78" y1="134.62" x2="-20.32" y2="134.62" width="0.1524" layer="91"/>
-<pinref part="X2" gate="G1" pin="5"/>
-<wire x1="-17.78" y1="137.16" x2="-20.32" y2="137.16" width="0.1524" layer="91"/>
-<wire x1="-20.32" y1="137.16" x2="-20.32" y2="135.89" width="0.1524" layer="91"/>
-<junction x="-20.32" y="135.89"/>
-<junction x="-20.32" y="134.62"/>
-<wire x1="-20.32" y1="133.35" x2="-20.32" y2="128.27" width="0.1524" layer="91"/>
-<pinref part="CC0" gate="G$1" pin="GND@3"/>
-<wire x1="-20.32" y1="128.27" x2="-25.4" y2="128.27" width="0.1524" layer="91"/>
-<junction x="-20.32" y="133.35"/>
-<pinref part="GND8" gate="1" pin="GND"/>
-<wire x1="-20.32" y1="125.73" x2="-20.32" y2="128.27" width="0.1524" layer="91"/>
-<junction x="-20.32" y="128.27"/>
-</segment>
-<segment>
 <pinref part="CC_X0" gate="G$1" pin="9"/>
 <wire x1="-49.53" y1="100.33" x2="-66.04" y2="100.33" width="0.1524" layer="91"/>
@@
 <net name="ANT" class="0">
 <segment>
-<pinref part="CC0" gate="G$1" pin="ANT"/>
-<pinref part="X2" gate="G1" pin="1"/>
-<wire x1="-25.4" y1="130.81" x2="-17.78" y2="130.81" width="0.1524" layer="91"/>
-<label x="-25.4" y="129.54" size="1.778" layer="95"/>
-</segment>
-<segment>
 <pinref part="RADIO0B" gate="G$1" pin="ANT"/>
 <wire x1="-25.4" y1="172.72" x2="-10.16" y2="172.72" width="0.1524" layer="91"/>
@@
 </segment>
 </net>
+<net name="N$3" class="0">
+<segment>
+<pinref part="X1" gate="G$1" pin="GND4"/>
+<pinref part="X1" gate="G$1" pin="GND3"/>
+<wire x1="-10.16" y1="123.19" x2="-15.24" y2="123.19" width="0.1524" layer="91"/>
+<wire x1="-15.24" y1="123.19" x2="-22.86" y2="123.19" width="0.1524" layer="91"/>
+<wire x1="-22.86" y1="123.19" x2="-22.86" y2="128.27" width="0.1524" layer="91"/>
+<pinref part="X1" gate="G$1" pin="GND2"/>
+<pinref part="X1" gate="G$1" pin="GND1"/>
+<wire x1="-10.16" y1="138.43" x2="-15.24" y2="138.43" width="0.1524" layer="91"/>
+<wire x1="-15.24" y1="138.43" x2="-22.86" y2="138.43" width="0.1524" layer="91"/>
+<wire x1="-22.86" y1="138.43" x2="-22.86" y2="133.35" width="0.1524" layer="91"/>
+<wire x1="-22.86" y1="133.35" x2="-22.86" y2="128.27" width="0.1524" layer="91"/>
+<junction x="-15.24" y="138.43"/>
+<junction x="-15.24" y="123.19"/>
+<pinref part="CC0" gate="G$1" pin="GND@2"/>
+<wire x1="-25.4" y1="133.35" x2="-22.86" y2="133.35" width="0.1524" layer="91"/>
+<pinref part="CC0" gate="G$1" pin="GND@3"/>
+<wire x1="-25.4" y1="128.27" x2="-22.86" y2="128.27" width="0.1524" layer="91"/>
+<junction x="-22.86" y="133.35"/>
+<junction x="-22.86" y="128.27"/>
+</segment>
+</net>
+<net name="N$1" class="0">
+<segment>
+<pinref part="CC0" gate="G$1" pin="ANT"/>
+<pinref part="X1" gate="G$1" pin="ANT"/>
+<wire x1="-25.4" y1="130.81" x2="-20.32" y2="130.81" width="0.1524" layer="91"/>
+</segment>
+</net>
