File: HW-MAPLE-Large/Archiv/V2.1/mapleCUx_large_210.brd (EAGLE design)
At the start: 100 x 59 mm, 66 parts, among them IC2 LAN-USR-ES1, IC31 ATMEGA168-TQFP, U1 RFM69HCW, X31 M03X2, X4 1751248, X7 1751264, Y2 8MHZ

Commit message: Docs V2.1
Parts:
- removed LED: (no value), led:CHIPLED_0805
- removed R32: 1k, rcl:R0805
- added C7: (no value), rcl:C1812
- X1, X2, X3, X5: device adafruit:SMA_EDGELAUNCH_UFL -> adafruit:SMA_EDGELAUNCH
- moved UART1 41.2 mm to (24.1, 55.9)
- moved DBG 17.7 mm to (35.6, 41.9), turned to 270 degrees
Connections:
- removed net M-SCK: X31.P$3
- removed net N$18: LED.A, R32.2
- removed net N$3: 3V3.2, 5V.1, F2.P$1
- removed net RX_LED: IC31.2, R32.1
- net +5V: now also C9.2, RS485.8
- net D13_SCK: now also X31.P$3
- net GND: now also C7.1; no longer LED.C
- net N$1: now also C7.2
- net RX-MAPLE: no longer U$2.RX1
- net TX-MAPLE: now also U$2.RX1
- net VCC: now also U$2.RAW
- net VDD: now also 3V3.2, 5V.1, F2.P$1; no longer C9.2, RS485.8
Routing:
- net TX-MAPLE: track 17.1 -> 73.2 mm, vias 0 -> 1
- net GND: track 680.4 -> 731.5 mm, vias 39 -> 3
- net CC_IN_0: track 58.9 -> 32.8 mm
- net D10_SS: track 61.2 -> 37.9 mm, vias 0 -> 3
- net CC_IN_1: track 84.2 -> 107.2 mm, vias 0 -> 3
- net D13_SCK: track 31.3 -> 52.2 mm, vias 0 -> 1
- net RX_DBG: track 85.3 -> 65.5 mm, vias 2 -> 1
- net SCK1: track 146.5 -> 165.4 mm, vias 3 -> 4
- net N$18: track 16.9 -> 0.00 mm, vias 1 -> 0
- net MISO1: track 150.3 -> 135.0 mm, vias 0 -> 2
- net N$19: track 25.5 -> 40.2 mm, vias 2 -> 0
- net TX_DBG: track 49.8 -> 35.1 mm
- net R1-HM: track 73.5 -> 61.2 mm
- net N$9: track 11.0 -> 0.13 mm
- net B: track 38.5 -> 48.8 mm
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Other:
- board text added: "MAPLE CUN"
- board text added: "MAPLE CUN - large -"
- board text added: "Version 2.1 www.neuby.de"
- board text removed: "MAPLE CUN - large"
- board text removed: "MAPLE CUN Large"
- board text removed: "Version 2.0 www.neuby.de"
