File: HW-MAPLE-Large/AddOns/1Wire-V01/Addon-mapleCUx_OneWire-RS485-007.brd (EAGLE design)
At the start: 67 x 47 mm, 36 parts, among them IC1 DS2482, IC31 ATMEGA168-TQFP, Q1 BSS84, X31 M03X2, X4 1751248, X7 1751264, Y2 8MHZ

Commit message: V3 Update + AddOns
V3 => 3.1 some more Cs

Addons:
-OneWire Beta
-RFM69: Module with other /  better Footprint
Parts:
- added EXT: (no value), jumper:SJ
- added R7, T2: (no value), jumper:SJ_2
- moved NRF24L01+ 33.0 mm to (55.9, 16.5)
- moved F1 25.9 mm to (62.2, 48.3), turned to 0 degrees
- moved R3 13.3 mm to (48.3, 44.5)
- moved Q1 13.0 mm to (38.1, 50.8)
- moved 3V3 10.9 mm to (41.9, 20.3)
- moved R4 7.62 mm to (87.6, 21.6), turned to 180 degrees
- moved GND 6.35 mm to (36.8, 20.3)
- moved ZD1 5.24 mm to (45.7, 53.3)
- moved 5V 5.08 mm to (41.9, 16.5)
- moved C14 5.08 mm to (95.2, 21.6), turned to 0 degrees
- moved IC1 4.58 mm to (43.2, 44.5)
- moved C31 4.58 mm to (95.2, 25.4), flipped to the top, turned to 0 degrees
- moved C32 4.58 mm to (90.2, 25.4), turned to 0 degrees
- moved R5 3.59 mm to (43.2, 36.8), turned to 0 degrees
- moved R10 2.84 mm to (61.0, 41.9)
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Connections:
- removed net R1-HM: R1.3
- removed net RX-MAPLE: U$1.TX0, UART0.3
- removed net T1-HM: T1.3
- removed net TX-MAPLE: U$1.RX1, UART0.2
- new net CE-M: IC31.13, NRF24L01+.3
- new net EXT: EXT.2, F1.P$1, R6.2, X7.1
- new net R1-ARD: R1.3, R7.3, U$1.TX0
- new net T1-ARD: T1.3, T2.3, U$1.RX1
- net CE-A: no longer IC31.13, NRF24L01+.3
- net CSN-A: no longer NRF24L01+.4
- net D10_SS: now also NRF24L01+.4
- net D11_MOSI: now also NRF24L01+.6
- net D12_MISO: now also NRF24L01+.7
- net D13_SCK: now also NRF24L01+.5
- net D2_INT0: now also NRF24L01+.8
- net IRQ-A: no longer NRF24L01+.8
- net MISO-A: no longer NRF24L01+.7
- net MOSI-A: no longer NRF24L01+.6
- net R1-MY: now also R7.1
- net RX1: now also R7.2, UART0.3
- net SCK-A: no longer NRF24L01+.5
- net T1-MY: now also T2.1
- net TX1: now also T2.2, UART0.2
- net VDD: now also EXT.1; no longer F1.P$1, R6.2, X7.1
Routing:
- net GND: track 0.00 -> 219.2 mm, vias 0 -> 15
- net VCC: track 0.00 -> 137.9 mm
- net VDD: track 0.00 -> 79.5 mm, vias 0 -> 1
- net GD: track 0.00 -> 75.8 mm
- net EXT: track 0.00 -> 69.2 mm, vias 0 -> 2
- net 1W: track 0.00 -> 55.1 mm, vias 0 -> 1
- net R1-MY: track 0.00 -> 52.9 mm
- net D13_SCK: track 0.00 -> 47.2 mm, vias 0 -> 1
- net D2_INT0: track 0.00 -> 47.2 mm, vias 0 -> 1
- net TX1: track 0.00 -> 45.9 mm
- net T1-MY: track 0.00 -> 44.6 mm
- net RX1: track 0.00 -> 41.4 mm
- net MOSI-A: track 0.00 -> 38.4 mm
- net 2W: track 0.00 -> 38.2 mm, vias 0 -> 1
- net D12_MISO: track 0.00 -> 37.1 mm, vias 0 -> 1
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- added copper zone on layer 1, net GND
- added copper zone on layer 16, net GND
