File: HW-MAPLE-Large/AddOns/RFM69-usw-V10/Addon-mapleCUx_HM-RFM69-V10-005.sch (EAGLE design)
At the start: 34 parts, among them IC1 ATSHA204A, IC31 ATMEGA168-TQFP, M2 NRF24L01+SMD, U1 RFM69HCW, X31 M03X2, X4 1751248, X7 1751264, Y2 8MHZ

Commit message: V3 Update + AddOns
V3 => 3.1 some more Cs

Addons:
-OneWire Beta
-RFM69: Module with other /  better Footprint
Parts:
- removed ANT: MICRO RF, SparkFun-Connectors:M01PTH
- removed M2: NRF24L01+SMD, wireless:NRF24L01+SMD
- removed R2: 10k, doug:RESISTOR0805-RES
- removed U1: RFM69HCW, doug:RFM69HCW
- removed X8: (no value), adafruit:SMACONNECTOR_EDGE
- added ANT1: (no value), pinhead:PINHD-1X1
- added EXT: (no value), jumper:SJ
- added R3: 10k, doug:RESISTOR0805-RES
- added RFM69W: RFM69HW, hoperf:RFM69HW
- added SJ1: (no value), jumper:SJ2W
- added X2: (no value), adafruit:SMACONNECTOR_EDGE
Connections:
- removed net 3.3V: M2.VCC
- removed net ANT: ANT.1, U1.ANT, X8.ANT
- removed net D7-ATSHA: IC1.SDA, IC31.PD7(AIN1)
- removed net N$14: U1.DIO2
- removed net N$15: U1.DIO1
- removed net N$16: U1.RESET
- new net D7-ATSHA-ARDU: SJ1.3, U$2.D7
- new net D7-ATSHA-MEGA: IC31.PD7(AIN1), SJ1.1
- new net EXT: EXT.2, F1.1, X7-1.K
- new net N$1: ANT1.1, RFM69W.ANT, X2.ANT
- new net N$5: IC1.SDA, SJ1.2
- net CE-A: now also U$2.D9; no longer M2.CE
- net CSN-A: now also R3.1, RFM69W.NSS; no longer R2.1, U1.NSS
- net D10_SS: no longer M2.CSN
- net D11_MOSI: no longer M2.MOSI
- net D12_MISO: no longer M2.MISO
- net D13_SCK: no longer M2.SCK
- net D2_INT0: no longer M2.IRQ
- net GND: now also RFM69W.GNDA, RFM69W.GNDB, X2.GND1, X2.GND2, X2.GND3, X2.GND4; no longer M2.GND, U1.GND_1, U1.GND_2, U1.GND_3, X8.GND1, X8.GND2, X8.GND3, X8.GND4
- net IRQ-A: now also RFM69W.DIO0; no longer U1.DIO0
- net MISO-A: now also RFM69W.MISO; no longer U1.MISO
- net MOSI-A: now also RFM69W.MOSI; no longer U1.MOSI
- net SCK-A: now also RFM69W.SCK; no longer U1.SCK
- net VCC: now also R3.2, RFM69W.VCC; no longer R2.2, U1.3.3V
- net VDD: now also EXT.1; no longer F1.1, X7-1.K
Other:
- note added: "Free Pins"
- note added: "Nur mit 3,3V Arduino!"
- note added: "RFM69(H)W"
- note removed: "Nrf24l01+ Radio"
- note removed: "because max. input voltage Vi = 5.25 V for NRF24L01+."
- note removed: "no resistor divider for CE necessary,"
