File: HW-MAPLE-Large/Archiv/V3.3/mapleCUx_large_330-014.brd (EAGLE design)
At the start: 100 x 59 mm, 34 parts, among them IC1 LD117ADT50TR, IC2 LAN-USR-ES1, IC6 LM1117MPX-ADJ

Commit message: V3.3 large
Parts:
- added NO_REGULATOR: JUMPER-SMT_2_NC_PASTE_NO-SILK, SparkFun-Jumpers:SMT-JUMPER_2_NC_PASTE_NO-SILK
- moved C1 14.9 mm to (25.0, 27.3), turned to 45 degrees
- moved CC0 14.0 mm to (32.1, 16.1), turned to 315 degrees
- moved U$2 1.27 mm to (0.25, 21.1)
Connections:
- net IN: now also NO_REGULATOR.2
- net VIN2: now also NO_REGULATOR.1
Routing:
- net MOSI1: track 140.0 -> 103.0 mm, vias 0 -> 2
- net SCK1: track 144.3 -> 108.7 mm, vias 0 -> 2
- net CC_CS0: track 68.0 -> 37.8 mm
- net MISO1: track 115.5 -> 139.0 mm
- net GND: track 587.4 -> 571.1 mm, vias 0 -> 2
- net CC_CS1: track 80.2 -> 94.4 mm, vias 2 -> 1
- net CC_OUT_0: track 51.2 -> 37.8 mm
- net CC_OUT_2: track 55.2 -> 43.2 mm
- net CC_IN_0: track 49.0 -> 37.8 mm
- net CC_CS2: track 53.7 -> 42.7 mm
- net VCC: track 260.0 -> 267.1 mm, vias 1 -> 2
- net VIN2: track 128.6 -> 122.7 mm
- net TX_DBG: track 72.7 -> 77.5 mm, vias 3 -> 2
- net CC_OUT_1: track 80.7 -> 85.1 mm, vias 0 -> 2
- net N$1: track 61.0 -> 57.9 mm
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Other:
- board text added: "Version 3.3 www.neuby.de"
- board text removed: "Version 3.2 www.neuby.de"
