File: HW-MAPLE-Large/AddOns/RasPi-UART__Zigbee-CC2530-V01/Addon-mapleCUx_Raspi-3V3-UART-CC2530-V007.brd (EAGLE design)
At the start: 49 x 47 mm, 15 parts, among them IC1 LD117ADT50TR, IC6 LM1117MPX-ADJ

Commit message: Raspi + Zigbee
Parts:
- removed HMMOD-UART: HM-MOD-UARTDIL, wireless:HM-MOD-UART-DIL
- added CC-DEBUG: (no value), con-lstb:MA05-2
- added EXT: (no value), jumper:SJ
- added F1: 1812L, ptc-littlefuse:1812L
- added RX_SEL1, TX_SEL1: JUMPER-SMT_3_1-NC_TRACE_SILK, SparkFun-Jumpers:SMT-JUMPER_3_1-NC_TRACE_SILK
- added U$3: CC2530_MODULE, Martin-Communication-V3:CC2530_DIL
- added X4: 1751248, con-phoenix-350:1751248
- moved C5 44.5 mm to (57.7, 27.4)
- moved C7 37.3 mm to (76.2, 19.1), turned to 0 degrees
- moved RX_SEL 26.5 mm to (72.4, 43.2), flipped to the bottom, turned to 180 degrees
- moved TX_SEL 24.4 mm to (72.4, 47.0), flipped to the bottom, turned to 180 degrees
- moved REGULATOR-USE 16.6 mm to (92.7, 41.9), flipped to the bottom, turned to 90 degrees
- moved C6 16.6 mm to (80.0, 36.2), turned to 90 degrees
- moved SV2 5.08 mm to (66.0, 17.8)
- moved C9 4.58 mm to (94.0, 49.5), flipped to the bottom
- moved SV1 4.58 mm to (59.7, 47.0)
- moved IC1 4.02 mm to (85.1, 49.5)
- moved IC6 3.81 mm to (86.4, 49.5)
Connections:
- new net CS: CC-DEBUG.5
- new net DC: CC-DEBUG.3, U$3.P2_2
- new net DD: CC-DEBUG.4, U$3.P2_1
- new net EXT: EXT.2, F1.P$1
- new net MISO: CC-DEBUG.10
- new net MOSI: CC-DEBUG.8
- new net N$2: RX_SEL1.2, U$3.P0_2\U_RX
- new net N$3: TX_SEL1.2, U$3.P0_3\U_TX
- new net N$45: F1.P$2, X4.1
- new net RST: CC-DEBUG.7, U$3.RST
- new net SCLK: CC-DEBUG.6
- new net VOLT-SENSE: CC-DEBUG.2
- net GND: now also CC-DEBUG.1, U$3.GND, U$3.GND2, X4.2; no longer HMMOD-UART.2
- net RX0: now also RX_SEL1.1
- net RX1: now also RX_SEL1.3; no longer HMMOD-UART.5
- net TX0: now also TX_SEL1.3
- net TX1: now also TX_SEL1.1; no longer HMMOD-UART.6
- net VCC: now also CC-DEBUG.9, EXT.1, U$3.VCC, U$3.VCC2; no longer HMMOD-UART.1
Routing:
- net N$3: track 0.00 -> 53.4 mm
- net N$2: track 0.00 -> 47.2 mm, vias 0 -> 1
- net TX1: track 75.2 -> 43.4 mm
- net VCC: track 131.3 -> 161.7 mm, vias 1 -> 0
- net DC: track 0.00 -> 27.9 mm
- net DD: track 0.00 -> 24.5 mm
- net RST: track 0.00 -> 18.9 mm
- net VIN2: track 46.6 -> 27.7 mm, vias 0 -> 1
- net RX1: track 66.9 -> 50.3 mm, vias 1 -> 2
- net TX: track 41.5 -> 25.7 mm, vias 1 -> 0
- net IN: track 30.8 -> 15.0 mm
- net GND: track 150.8 -> 166.3 mm
- net RX0: track 54.0 -> 60.2 mm
- net N$45: track 0.00 -> 5.45 mm
- net EXT: track 0.00 -> 3.86 mm
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