File: HW-MAPLE-Large/AddOns/RasPi-UART__Zigbee-CC2530/Addon-mapleCUx_Raspi-3V3-UART-CC2530-V02-03.brd (EAGLE design)
At the start: 49 x 47 mm, 23 parts, among them IC1 LD117ADT50TR, IC6 LM1117MPX-ADJ, X4 1751248

Commit message: V3.4
Parts:
- U$3: device Martin-Communication-V3:CC2530_DIL -> Martin-Communication-V4:CC2530_DIL
- moved TX_SEL1 39.3 mm to (42.6, 2.05)
- moved TX_SEL 3.00 mm to (21.4, 32.0)
- moved REGULATOR-USE 2.43 mm to (39.3, 30.1), turned to 270 degrees
- moved RX_SEL 2.00 mm to (21.4, 29.2)
- moved RX_SEL1 1.50 mm to (3.39, 1.76), turned to 180 degrees
- moved EXT 1.41 mm to (45.8, 23.3)
- moved REBOOT 1.00 mm to (44.2, 42.9)
Connections:
- net TX0: now also TX_SEL.1, TX_SEL1.3; no longer TX_SEL.3, TX_SEL1.1
- net TX1: now also TX_SEL.3, TX_SEL1.1; no longer TX_SEL.1, TX_SEL1.3
Routing:
- net TX1: track 42.5 -> 91.2 mm
- net N$3: track 58.0 -> 17.1 mm, vias 1 -> 0
- net IN2: track 65.1 -> 53.4 mm, vias 0 -> 1
- net N$1: track 51.9 -> 42.1 mm
- net TX0: track 57.0 -> 65.9 mm
- net VCC: track 171.2 -> 162.9 mm
- net DC: track 27.9 -> 36.2 mm, vias 0 -> 1
- net IN: track 31.0 -> 38.7 mm
- net GND: track 174.8 -> 180.3 mm
- net RX: track 32.6 -> 27.1 mm
- net N$2: track 45.8 -> 50.5 mm, vias 1 -> 0
- net DD: track 24.5 -> 28.8 mm, vias 0 -> 1
- net RX0: track 59.1 -> 61.1 mm
- net TX: track 25.7 -> 23.7 mm
- net RX1: track 51.1 -> 51.0 mm, vias 1 -> 2
Other:
- board text added: "for 3V3 Serial Raspi AddOns and CC2530 V0.2"
- board text added: "older Board dont have 5 Pins =>"
- board text removed: "for 3V3 Serial Raspi AddOns and CC2530 V0.1"
