File: HW-MAPLE-Large/AddOns/RasPi-UART__Zigbee-CC2530/Addon-mapleCUx_Raspi-3V3-UART-CC2530-V02-03.sch (EAGLE design)
At the start: 23 parts, among them IC1 LD117ADT50TR, IC6 LM1117MPX-ADJ, X4 1751248

Commit message: V3.4
Connections:
- net TX0: now also TX_SEL.1; no longer TX_SEL.3
- net TX1: now also TX_SEL.3; no longer TX_SEL.1
Changed lines of the file:
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@@
-</segment>
-<segment>
-<pinref part="TX_SEL" gate="G$1" pin="1"/>
-<wire x1="20.32" y1="-111.76" x2="27.94" y2="-111.76" width="0.1524" layer="91"/>
-<label x="27.94" y="-111.76" size="1.778" layer="95"/>
 </segment>
 <segment>
@@
 <wire x1="182.88" y1="-154.94" x2="190.5" y2="-154.94" width="0.1524" layer="91"/>
 <label x="190.5" y="-154.94" size="1.778" layer="95"/>
+</segment>
+<segment>
+<pinref part="TX_SEL" gate="G$1" pin="3"/>
+<wire x1="20.32" y1="-121.92" x2="27.94" y2="-121.92" width="0.1524" layer="91"/>
+<label x="27.94" y="-121.92" size="1.778" layer="95"/>
 </segment>
 </net>
@@
 <net name="TX0" class="0">
 <segment>
-<pinref part="TX_SEL" gate="G$1" pin="3"/>
-<wire x1="20.32" y1="-121.92" x2="27.94" y2="-121.92" width="0.1524" layer="91"/>
-<label x="27.94" y="-121.92" size="1.778" layer="95"/>
-</segment>
-<segment>
 <pinref part="UART0" gate="1" pin="2"/>
 <wire x1="154.94" y1="-44.45" x2="143.51" y2="-44.45" width="0.1524" layer="91"/>
@@
 <label x="190.5" y="-165.1" size="1.778" layer="95"/>
 </segment>
+<segment>
+<pinref part="TX_SEL" gate="G$1" pin="1"/>
+<wire x1="20.32" y1="-111.76" x2="27.94" y2="-111.76" width="0.1524" layer="91"/>
+<label x="27.94" y="-111.76" size="1.778" layer="95"/>
+</segment>
 </net>
