File: HW-MAPLE-Large/AddOns/RasPi-UART__Zigbee-CC2530/Addon-mapleCUx_Raspi-3V3-UART-CC2530-V02-05.sch (EAGLE design)
At the start: 23 parts, among them IC1 LD117ADT50TR, IC6 LM1117MPX-ADJ, X4 1751248

Commit message: Zigbee
Parts:
- removed REBOOT: (no value), pinhead:PINHD-1X2
- removed REGULATOR-USE: JUMPER-SMT_3_1-NC_TRACE_SILK, SparkFun-Jumpers:JUMPER-SMT_3_1-NC_TRACE_SILK
- added AIR602: (no value), AIR602:AIR602
- added BOOT, REG1: (no value), jumper:SJ
- added C2: 22pF, rcl:C-EUC0805
- added E1: ANTENNA-GROUNDEDTRACE-25.7MM, SparkFun-RF:ANTENNA-GROUNDEDTRACE-25.7MM
- added U.FL: U.FL, SparkFun-Connectors:U.FL
- renumbered EXT to REG, RX_SEL1 to TX_1, TX_SEL1 to RX_1
Connections:
- removed net R: DBG.4
- removed net T: DBG.3
- removed net VIN2: REGULATOR-USE.1
- removed net VOLT-SENSE: CC-DEBUG.2
- new net N$4: AIR602.ANT, E1.SIGNAL, U.FL.SIGNAL
- new net RX_DBG: AIR602.TX1, DBG.4
- new net TX_DBG: AIR602.RX1, DBG.3
- net GND: now also AIR602.GND1, AIR602.GND2, BOOT.1, C2.1, E1.GND, U.FL.GND@0, U.FL.GND@1; no longer REBOOT.1
- net IN: now also REG1.1; no longer REGULATOR-USE.3
- net N$1: now also BOOT.2; no longer REBOOT.2
- net RX0: now also RX_1.3; no longer TX_1.3
- net RX1: now also RX_1.1; no longer TX_1.1
- net TX0: now also TX_1.3; no longer RX_1.3
- net TX1: now also TX_1.1; no longer RX_1.1
- net VCC: now also AIR602.VCC, C2.2, CC-DEBUG.2, REG1.2; no longer REGULATOR-USE.2
Other:
- note added: "AIR602 from Seeed"
- note added: "Volt-Sense"
- note removed: "könnte weg"
