File: HW-MAPLE-Large/Archiv/V3.4/mapleCUx_large_340-007.brd (EAGLE design)
At the start: 100 x 59 mm, 34 parts, among them IC1 LD117ADT50TR, IC2 LAN-USR-ES1, IC6 LM1117MPX-ADJ

Commit message: Zigbee
Routing:
- net N$4: track 2.39 -> 3.61 mm
Other:
- board text added: "Ant4"
- board text added: "C7"
- board text added: "Fuse"
- board text added: "Socket CC1101 TRX. 3"
- board text added: "U.FL"
- board text added: "cut Antenna here"
- board text removed: "Ant0"
- board text removed: "CC3"
- board text removed: "Socket CC1101 Transc. 2+3"
