File: HW-MAPLE-Large/Archiv/V3.5/mapleCUx_large_350-010.brd (EAGLE design)
At the start: 100 x 59 mm, 41 parts, among them IC1 LD117ADT50TR, IC2 LAN-USR-ES1, IC3 DS2482, IC6 LM1117MPX-ADJ, Q1 BSS84

Commit message: V3.5 and 1W Stamp
Parts:
- removed GND: (no value), jumper:SJ
- removed IC1: LD117ADT50TR, v-reg:DPACK
- added 1117: LD117ADT50TR, v-reg:DPACK
- moved NO_REGULATOR 19.0 mm to (37.5, 17.8), turned to 180 degrees
- moved JP1 15.7 mm to (21.6, 1.91), turned to 180 degrees
- moved IC6 14.8 mm to (37.5, 12.1), turned to 180 degrees
- moved R2 7.65 mm to (26.0, 17.1), turned to 180 degrees
- moved F1 4.49 mm to (18.2, 21.3)
- moved NO_FUSE 4.49 mm to (18.2, 21.6)
- moved C9 4.09 mm to (19.1, 17.1), turned to 180 degrees
- moved Q1 4.07 mm to (29.2, 10.8), turned to 0 degrees
- moved IC3 2.29 mm to (21.6, 11.4)
- moved ZD1 2.01 mm to (11.4, 8.89)
- moved R1 1.91 mm to (19.7, 5.08)
- moved R4 1.91 mm to (24.8, 5.08)
Connections:
- net 1W-GND: no longer GND.2
- net GND: now also 1117.1; no longer GND.1, IC1.1
- net IN: now also 1117.3, CC2-EXT.5; no longer IC1.3
- net VIN2: now also 1117.4; no longer IC1.4
Routing:
- net IN: track 26.1 -> 78.0 mm, vias 0 -> 3
- net GND: track 580.5 -> 547.2 mm, vias 3 -> 41
- net SWCLK/TCK: track 77.2 -> 101.3 mm, vias 0 -> 2
- net 1W-GND: track 96.2 -> 73.1 mm
- net CC_CS2: track 109.5 -> 87.6 mm, vias 2 -> 1
- net MISO1: track 120.5 -> 101.9 mm
- net SCK1: track 120.5 -> 106.1 mm
- net RX1: track 58.8 -> 72.8 mm
- net CC_CS0: track 43.7 -> 30.4 mm
- net CC_IN_2: track 98.5 -> 87.2 mm, vias 5 -> 1
- net MOSI1: track 119.2 -> 109.3 mm, vias 3 -> 1
- net NRESET: track 53.1 -> 63.0 mm, vias 0 -> 1
- net CC_OUT_2: track 74.5 -> 84.3 mm, vias 1 -> 3
- net WIZ_RST: track 31.0 -> 39.7 mm, vias 1 -> 0
- net CC_IN_3: track 67.5 -> 75.9 mm, vias 2 -> 1
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Other:
- board text added: "1W"
- board text added: "BSS84"
- board text added: "C9"
- board text added: "CLK"
- board text added: "DIO"
- board text added: "DS2482"
- board text added: "R1"
- board text added: "R2"
- board text added: "R4"
- board text added: "Version 3.5 www.neuby.de"
- board text removed: "Version 3.4b www.neuby.de"
