File: HW-MAPLE-Large/Archiv/V3.5/mapleCUx_large_350-010.sch (EAGLE design)
At the start: 41 parts, among them IC1 LD117ADT50TR, IC2 LAN-USR-ES1, IC3 DS2482, IC6 LM1117MPX-ADJ, Q1 BSS84

Commit message: V3.5 and 1W Stamp
Parts:
- removed GND: (no value), jumper:SJ
- renumbered IC1 to 1117
Connections:
- net 1W-GND: no longer GND.2
- net GND: no longer GND.1
- net IN: now also CC2-EXT.5V
