File: HW-MAPLE-Large/AddOns/Addon-LAN-WLAN-without-MAPLE/Addon-LAN-WLAN-without-MAPLE_or-OneWire_or_RS485-V01-010.sch (EAGLE design)
At the start: 32 parts, among them IC1 LD117ADT50TR, IC2 DS2480B, IC6 LM1117MPX-ADJ, M1 ARDUINO-PRO-MINI-3.3V#NP, X4 1751248, X7 1751264

Commit message: 1W-UART
Parts:
- removed SJ3, SJ4: (no value), jumper:SJ2W
- added RX, TX: (no value), jumper:SJ2W
- NOREG: value (none) -> JUMPER-SMT_2_NC_PASTE_NO-SILK; device jumper:SJ -> SparkFun-Jumpers:JUMPER-SMT_2_NC_PASTE_NO-SILK
- R4: value 150R -> 5K6
- R5: value 330R -> 22K
- R6: value 330R -> 4K7
Connections:
- net A: now also R4.2; no longer R4.1
- net B: no longer R4.2
- net D8: now also RX.3; no longer SJ3.3
- net D9: now also TX.3; no longer SJ4.3
- net DI1: now also TX.2; no longer SJ4.2
- net GND: now also R4.1
- net IN: now also R5.1
- net RO: now also RX.2; no longer SJ3.2
- net RX: now also RX.1; no longer SJ3.1
- net TX: now also TX.1; no longer SJ4.1
- net VCC: no longer R5.1
Other:
- note added: "Conectors to AddOn- or Main-PCB"
- note added: "OneWire (or RS485 Connections)"
- note added: "Power"
- note added: "RS485 Arduino"
- note added: "USR-TCP232-E2 or hopefully T2"
- note removed: "1 3V3 6 GND 8 TXD 9 GND 10 RXD"
- moved on the sheet: C10, R4, R5, R6, RAW, RS485, RX_1, RX_SEL, TX_1, TX_SEL
