File: HW-MAPLE-Large/AddOns/Addon-LAN-WLAN-without-MAPLE/Addon-LAN-WLAN-without-MAPLE_or-OneWire_or_RS485-V01-012.sch (EAGLE design)
At the start: 32 parts, among them IC1 LD117ADT50TR, IC2 DS2480B, IC6 LM1117MPX-ADJ, M1 ARDUINO-PRO-MINI-3.3V#NP, X4 1751248, X7 1751264

Commit message: OneWire
Connections:
- new net VINPUT: F1.2, NOFUSE.2, U$2.TIP, X4-1.K
- net IN: no longer C9.1, F1.1, IC1.IN, IC6.IN, NOFUSE.1, NOREG.2
- net VIN: now also C9.1, F1.1, IC1.IN, IC6.IN, NOFUSE.1, NOREG.2; no longer F1.2, NOFUSE.2, U$2.TIP, X4-1.K
