File: HW-MAPLE-Large/V4.0/mapleCUx_large_400-003.brd (EAGLE design)
At the start: 100 x 59 mm, 40 parts, among them IC2 LAN-USR-ES1, IC3 DS2482, IC6 LM1117MPX-ADJ, Q1 BSS84

Commit message: V4 first draft
Parts:
- removed DBG: (no value), con-lstb:MA05-1
- removed UART0, UART1: (no value), con-lstb:MA04-1
- added U$3, U$4: MAPLE-CUL-ADDON-V01, Martin-Communication-V4:MAPLE-CUL-V01
- moved C5 30.6 mm to (50.7, 28.4), turned to 90 degrees
- moved C7 20.1 mm to (28.1, 28.6), turned to 180 degrees
- moved CHPD1 7.94 mm to (71.4, 41.9)
- moved WLAN 7.62 mm to (71.1, 43.9)
- moved CC3 5.68 mm to (60.8, 25.8), turned to 260 degrees
- moved CC2 1.52 mm to (35.7, 26.3), turned to 255 degrees
- moved C12 0.51 mm to (84.6, 41.1)
- moved CC1 0.51 mm to (80.5, 24.8)
Connections:
- net GND: now also C9.1, U$3.GND, U$3.GND1, U$4.GND, U$4.GND1; no longer C9.2, DBG.5, UART0.4, UART1.4
- net IN: now also C9.2; no longer C9.1
- net RX-MAPLE: now also U$3.RX-MAP, U$4.RX-MAP; no longer UART0.3
- net RX1: now also U$3.RX-MAP1; no longer UART1.3
- net RX_DBG: now also U$4.RX-MAP1; no longer DBG.4
- net TX-MAPLE: now also U$3.TX-MAP, U$4.TX-MAP; no longer UART0.2
- net TX1: now also U$3.TX-MAP1; no longer UART1.2
- net TX_DBG: now also U$4.TX-MAP1; no longer DBG.3
- net VCC: now also U$3.VCC, U$3.VCC1, U$4.VCC, U$4.VCC1; no longer DBG.2, UART0.1, UART1.1
- net VIN2: no longer DBG.1
Routing:
- net GND: track 547.2 -> 0.00 mm, vias 41 -> 0
- net VCC: track 259.6 -> 0.00 mm, vias 1 -> 0
- net VIN2: track 127.8 -> 0.00 mm, vias 1 -> 0
- net MOSI1: track 109.3 -> 0.00 mm, vias 1 -> 0
- net SCK1: track 106.1 -> 0.00 mm, vias 2 -> 0
- net MISO1: track 101.9 -> 0.00 mm, vias 3 -> 0
- net SWCLK/TCK: track 101.3 -> 0.00 mm, vias 2 -> 0
- net CC_IN_1: track 100.0 -> 0.00 mm, vias 2 -> 0
- net CC_OUT_1: track 88.2 -> 0.00 mm
- net CC_CS2: track 87.6 -> 0.00 mm, vias 1 -> 0
- net CC_IN_2: track 87.2 -> 0.00 mm, vias 1 -> 0
- net CC_OUT_2: track 84.3 -> 0.00 mm, vias 3 -> 0
- net CC_CS1: track 84.0 -> 0.00 mm, vias 2 -> 0
- net RX_DBG: track 82.6 -> 0.00 mm, vias 2 -> 0
- net SWDIO/TMS: track 78.2 -> 0.00 mm, vias 2 -> 0
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