File: HW-MAPLE-Large/V4.0/mapleCUx_large_400-003.sch (EAGLE design)
At the start: 40 parts, among them IC2 LAN-USR-ES1, IC3 DS2482, IC6 LM1117MPX-ADJ, Q1 BSS84

Commit message: V4 first draft
Parts:
- removed DBG: (no value), con-lstb:MA05-1
- removed UART0, UART1: (no value), con-lstb:MA04-1
- added U$3, U$4: MAPLE-CUL-ADDON-V01, Martin-Communication-V4:MAPLE-CUL-ADDON-V01
Connections:
- net GND: now also C9.1, U$3.GND, U$3.GND1, U$4.GND, U$4.GND1; no longer C9.2, DBG.5, UART0.4, UART1.4
- net IN: now also C9.2; no longer C9.1
- net RX-MAPLE: now also U$3.RX-MAPLE, U$4.RX-MAPLE; no longer UART0.3
- net RX1: now also U$3.RX-MAPLE1; no longer UART1.3
- net RX_DBG: now also U$4.RX-MAPLE1; no longer DBG.4
- net TX-MAPLE: now also U$3.TX-MAPLE, U$4.TX-MAPLE; no longer UART0.2
- net TX1: now also U$3.TX-MAPLE1; no longer UART1.2
- net TX_DBG: now also U$4.TX-MAPLE1; no longer DBG.3
- net VCC: now also U$3.VCC, U$3.VCC1, U$4.VCC, U$4.VCC1; no longer DBG.2, UART0.1, UART1.1
- net VIN2: no longer DBG.1
Other:
- note added: "1W: Alternativ als Steckmodul"
- note added: "Debug"
- note added: "UART0"
- note added: "UART1"
- note removed: "1Wire"
- note removed: "Opt"
- note removed: "siehe Homematic"
- note removed: "siehe MySensors"
- moved on the sheet: 1117, C9, CC2-EXT, F1, IC3, IC6, J2, JP1, NO_FUSE, NO_REGULATOR, PROG, Q1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
