File: HW-MAPLE-Large/V4.0/mapleCUx_large_400-012.brd (EAGLE design)
At the start: 100 x 59 mm, 39 parts, among them IC2 LAN-USR-ES1, IC3 DS2482, IC6 LM1117MPX-ADJ, Q1 BSS84

Commit message: V4
Parts:
- removed CC2-EXT: ONEWIRE-MODULE, CC1101:ONEWIRE_CC1101_MODULE3_DIL
- added CC3-EXT: ONEWIRE-MODULE, CC1101:ONEWIRE_CC1101_MODULE3_DIL
- moved X1 76.8 mm to (10.2, 0.00)
- moved X5 76.8 mm to (87.0, 0.00)
- moved CC1 64.8 mm to (15.7, 26.0), turned to 250 degrees
- moved CC0 64.2 mm to (80.5, 24.6), turned to 270 degrees
- moved U$3 31.8 mm to (52.7, 8.26)
- moved U$4 27.3 mm to (99.7, 50.8)
- moved CC3 26.7 mm to (34.2, 25.8)
- moved X2 25.4 mm to (61.0, 0.00)
- moved X3 25.4 mm to (35.6, 0.00)
- moved CC2 24.1 mm to (59.8, 25.7), turned to 260 degrees
- moved VTRX2 22.0 mm to (72.5, 20.2), turned to 180 degrees
- moved C7 21.0 mm to (7.11, 26.7)
- moved NO_REGULATOR 17.1 mm to (20.3, 17.8), turned to 90 degrees
- moved C9 15.6 mm to (22.2, 1.91)
- moved R1 15.5 mm to (34.9, 7.62), turned to 270 degrees
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Connections:
- net 1W: now also CC3-EXT.1W; no longer CC2-EXT.1W
- net 1W-GND: now also CC3-EXT.1W-GND; no longer CC2-EXT.1W-GND
- net CC_CS2: now also CC3-EXT.CSN; no longer CC2-EXT.CSN
- net CC_IN_2: now also CC3-EXT.GDO2; no longer CC2-EXT.GDO2
- net CC_OUT_2: now also CC3-EXT.GDO0; no longer CC2-EXT.GDO0
- net GND: now also CC3-EXT.GND@0, CC3-EXT.GND@1; no longer CC2-EXT.GND@0, CC2-EXT.GND@1
- net IN: now also CC3-EXT.5; no longer CC2-EXT.5
- net MISO1: now also CC3-EXT.MISO; no longer CC2-EXT.MISO
- net MOSI1: now also CC3-EXT.MOSI; no longer CC2-EXT.MOSI
- net RX-MAPLE: now also HMMOD-UART.5
- net RX1: no longer HMMOD-UART.5
- net SCK1: now also CC3-EXT.SCK; no longer CC2-EXT.SCK
- net TX-MAPLE: now also HMMOD-UART.6
- net TX1: no longer HMMOD-UART.6
- net VCC: now also CC3-EXT.VCC@0, CC3-EXT.VCC@1; no longer CC2-EXT.VCC@0, CC2-EXT.VCC@1
Routing:
- net GND: track 0.00 -> 505.8 mm, vias 0 -> 43
- net VCC: track 0.00 -> 277.9 mm
- net TX-MAPLE: track 0.00 -> 140.6 mm, vias 0 -> 1
- net MOSI1: track 0.00 -> 127.9 mm, vias 0 -> 2
- net CC_IN_2: track 0.00 -> 123.7 mm, vias 0 -> 2
- net CC_CS2: track 0.00 -> 109.4 mm, vias 0 -> 1
- net MISO1: track 0.00 -> 108.9 mm, vias 0 -> 1
- net RX-MAPLE: track 0.00 -> 107.7 mm, vias 0 -> 2
- net SCK1: track 0.00 -> 102.8 mm, vias 0 -> 2
- net CC_OUT_0: track 0.00 -> 87.8 mm, vias 0 -> 1
- net 1W: track 0.00 -> 86.7 mm
- net TX1: track 0.00 -> 85.5 mm
- net CC_IN_0: track 0.00 -> 82.9 mm, vias 0 -> 2
- net 1W-GND: track 0.00 -> 82.8 mm
- net SWCLK/TCK: track 0.00 -> 80.2 mm
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Other:
- board text added: "1Wire"
- board text added: "DBG"
- board text added: "MAPLE CUL"
- board text added: "MAPLE CUL - large -"
- board text added: "Socket TRX3"
- board text added: "UART1"
- board text added: "UART2"
- board text added: "Version 4.0 www.neuby.de"
- board text removed: "C7"
- board text removed: "MAPLE CUN"
- board text removed: "MAPLE CUN - large -"
- board text removed: "R"
- board text removed: "RX"
- board text removed: "Socket CC1101 TRX. 3"
- board text removed: "T"
- board text removed: "TX"
- board text removed: "VIN"
- board text removed: "Version 3.5 www.neuby.de"
- board text removed: "WLAN from Seeedstudio..."
