File: HW-MAPLE-Large/V4.0/mapleCUx_large_401-014-not-produced.sch (EAGLE design)
At the start: 40 parts, among them IC2 LAN-USR-ES1, IC3 DS2482, IC6 LM1117MPX-ADJ, Q1 BSS84

Commit message: Fix for old RFM69 AddOn + Docu
Parts:
- removed CC2-EXT: ONEWIRE-MODULE, CC1101:ONEWIRE-MODULE
- removed DBG: (no value), con-lstb:MA05-1
- removed UART0, UART1: (no value), con-lstb:MA04-1
- added CC3-EXT: ONEWIRE-MODULE, CC1101:ONEWIRE-MODULE
- added U$3, U$4: MAPLE-CUL-ADDON-V01, Martin-Communication-V4:MAPLE-CUL-ADDON-V01
Connections:
- net 1W: now also CC3-EXT.1W; no longer CC2-EXT.1W
- net 1W-GND: now also CC3-EXT.1W-GND; no longer CC2-EXT.1W-GND
- net CC_CS2: now also CC3-EXT.CSN; no longer CC2-EXT.CSN
- net CC_IN_2: now also CC3-EXT.GDO2; no longer CC2-EXT.GDO2
- net CC_OUT_2: now also CC3-EXT.GDO0; no longer CC2-EXT.GDO0
- net GND: now also C9.1, CC3-EXT.GND@0, CC3-EXT.GND@1, U$3.GND, U$3.GND1, U$4.GND, U$4.GND1; no longer C9.2, CC2-EXT.GND@0, CC2-EXT.GND@1, DBG.5, UART0.4, UART1.4
- net IN: now also C9.2, CC3-EXT.5V; no longer C9.1, CC2-EXT.5V
- net MISO1: now also CC3-EXT.MISO; no longer CC2-EXT.MISO
- net MOSI1: now also CC3-EXT.MOSI; no longer CC2-EXT.MOSI
- net RX-MAPLE: now also HMMOD-UART.TX, U$3.RX-MAPLE, U$4.RX-MAPLE; no longer UART0.3
- net RX1: now also U$3.RX-MAPLE1; no longer HMMOD-UART.TX, UART1.3
- net RX_DBG: now also U$4.RX-MAPLE1; no longer DBG.4
- net SCK1: now also CC3-EXT.SCLK; no longer CC2-EXT.SCLK
- net TX-MAPLE: now also HMMOD-UART.RX, U$3.TX-MAPLE, U$4.TX-MAPLE; no longer UART0.2
- net TX1: now also U$3.TX-MAPLE1; no longer HMMOD-UART.RX, UART1.2
- net TX_DBG: now also U$4.TX-MAPLE1; no longer DBG.3
- net VCC: now also CC3-EXT.VCC@0, CC3-EXT.VCC@1, U$3.VCC, U$3.VCC1, U$4.VCC, U$4.VCC1; no longer CC2-EXT.VCC@0, CC2-EXT.VCC@1, DBG.2, UART0.1, UART1.1
- net VIN2: no longer DBG.1
Other:
- note added: "1W: Alternativ als Steckmodul"
- note added: "Debug"
- note added: "UART0"
- note added: "UART1"
- note removed: "1Wire"
- note removed: "Opt"
- note removed: "siehe Homematic"
- note removed: "siehe MySensors"
- moved on the sheet: 1117, C9, F1, IC3, IC6, J2, JP1, NO_FUSE, NO_REGULATOR, PROG, Q1, R1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
