File: HW-MAPLE-Large/V4.0/mapleCUx_large_4.1-018-not-produced.sch (EAGLE design)
At the start: 39 parts, among them IC2 LAN-USR-ES1, IC3 DS2482, IC6 LM1117MPX-ADJ, Q1 BSS84

Commit message: V4 General Update
Connections:
- net RX-MAPLE: now also U$3.RX-MAPLE1; no longer U$3.RX-MAPLE
- net RX1: now also U$3.RX-MAPLE; no longer U$3.RX-MAPLE1
- net TX-MAPLE: now also U$3.TX-MAPLE1; no longer U$3.TX-MAPLE
- net TX1: now also U$3.TX-MAPLE; no longer U$3.TX-MAPLE1
- net VIN2: now also U$3.5V, U$4.5V
Other:
- note added: "5V Tolererant"
Changed lines of the file:
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@@
 <?xml version="1.0" encoding="utf-8"?>
 <!DOCTYPE eagle SYSTEM "eagle.dtd">
-<eagle version="9.3.0">
+<eagle version="9.1.1">
 <drawing>
 <settings>
@@
 <text x="190.5" y="67.31" size="1.778" layer="95">UART1</text>
 <text x="143.51" y="68.58" size="1.778" layer="95">UART0</text>
+<text x="193.04" y="113.03" size="1.778" layer="97">5V Tolererant</text>
 </plain>
 <instances>
@@
 <attribute name="VALUE" x="63.5" y="12.7" size="1.778" layer="96"/>
 </instance>
-<instance part="SUPPLY13" gate="G$1" x="129.54" y="78.74" smashed="yes">
-<attribute name="VALUE" x="127.635" y="81.915" size="1.778" layer="96"/>
+<instance part="SUPPLY13" gate="G$1" x="129.54" y="76.2" smashed="yes">
+<attribute name="VALUE" x="127.635" y="79.375" size="1.778" layer="96"/>
 </instance>
 <instance part="SUPPLY14" gate="G$1" x="214.63" y="60.96" smashed="yes" rot="R270">
@@
 <segment>
 <pinref part="U$3" gate="G$1" pin="VCC"/>
-<wire x1="137.16" y1="76.2" x2="129.54" y2="76.2" width="0.1524" layer="91"/>
-<wire x1="129.54" y1="76.2" x2="129.54" y2="45.72" width="0.1524" layer="91"/>
+<wire x1="137.16" y1="73.66" x2="129.54" y2="73.66" width="0.1524" layer="91"/>
+<wire x1="129.54" y1="73.66" x2="129.54" y2="43.18" width="0.1524" layer="91"/>
 <pinref part="U$4" gate="G$1" pin="VCC"/>
-<wire x1="129.54" y1="45.72" x2="137.16" y2="45.72" width="0.1524" layer="91"/>
+<wire x1="129.54" y1="43.18" x2="137.16" y2="43.18" width="0.1524" layer="91"/>
 <pinref part="SUPPLY13" gate="G$1" pin="VCC"/>
-<junction x="129.54" y="76.2"/>
+<junction x="129.54" y="73.66"/>
 </segment>
 <segment>
@@
 </segment>
 <segment>
-<pinref part="U$3" gate="G$1" pin="RX-MAPLE1"/>
-<wire x1="203.2" y1="71.12" x2="219.71" y2="71.12" width="0.1524" layer="91"/>
-<label x="219.71" y="71.12" size="1.778" layer="95" xref="yes"/>
+<pinref part="U$3" gate="G$1" pin="RX-MAPLE"/>
+<wire x1="137.16" y1="66.04" x2="114.3" y2="66.04" width="0.1524" layer="91"/>
+<label x="114.3" y="66.04" size="1.778" layer="95" rot="R180" xref="yes"/>
 </segment>
 </net>
@@
 </segment>
 <segment>
-<pinref part="U$3" gate="G$1" pin="TX-MAPLE1"/>
-<wire x1="203.2" y1="66.04" x2="219.71" y2="66.04" width="0.1524" layer="91"/>
-<label x="219.71" y="66.04" size="1.778" layer="95" xref="yes"/>
+<pinref part="U$3" gate="G$1" pin="TX-MAPLE"/>
+<wire x1="137.16" y1="71.12" x2="114.3" y2="71.12" width="0.1524" layer="91"/>
+<label x="114.3" y="71.12" size="1.778" layer="95" rot="R180" xref="yes"/>
 </segment>
 </net>
@@
 </segment>
 <segment>
-<pinref part="U$3" gate="G$1" pin="RX-MAPLE"/>
-<wire x1="137.16" y1="66.04" x2="114.3" y2="66.04" width="0.1524" layer="91"/>
-<label x="114.3" y="66.04" size="1.778" layer="95" rot="R180" xref="yes"/>
-</segment>
-<segment>
 <pinref part="HMMOD-UART" gate="G$1" pin="TX"/>
 <wire x1="317.5" y1="76.2" x2="297.18" y2="76.2" width="0.1524" layer="91"/>
 <label x="302.26" y="76.2" size="1.778" layer="95"/>
 </segment>
+<segment>
+<pinref part="U$3" gate="G$1" pin="RX-MAPLE1"/>
+<wire x1="203.2" y1="71.12" x2="219.71" y2="71.12" width="0.1524" layer="91"/>
+<label x="219.71" y="71.12" size="1.778" layer="95" xref="yes"/>
+</segment>
 </net>
 <net name="TX-MAPLE" class="0">
@@
 </segment>
 <segment>
-<pinref part="U$3" gate="G$1" pin="TX-MAPLE"/>
-<wire x1="137.16" y1="71.12" x2="114.3" y2="71.12" width="0.1524" layer="91"/>
-<label x="114.3" y="71.12" size="1.778" layer="95" rot="R180" xref="yes"/>
-</segment>
-<segment>
 <pinref part="HMMOD-UART" gate="G$1" pin="RX"/>
 <wire x1="317.5" y1="78.74" x2="297.18" y2="78.74" width="0.1524" layer="91"/>
 <label x="302.26" y="78.74" size="1.778" layer="95"/>
+</segment>
+<segment>
+<pinref part="U$3" gate="G$1" pin="TX-MAPLE1"/>
+<wire x1="203.2" y1="66.04" x2="219.71" y2="66.04" width="0.1524" layer="91"/>
+<label x="219.71" y="66.04" size="1.778" layer="95" xref="yes"/>
 </segment>
 </net>
@@
 <label x="351.79" y="176.53" size="1.778" layer="95" rot="R180" xref="yes"/>
 </segment>
-</net>
+<segment>
+<pinref part="U$3" gate="G$1" pin="5V"/>
+<wire x1="137.16" y1="76.2" x2="137.16" y2="81.28" width="0.1524" layer="91"/>
+<label x="137.16" y="81.28" size="1.778" layer="95" rot="R90" xref="yes"/>
+</segment>
+<segment>
+<pinref part="U$4" gate="G$1" pin="5V"/>
+<wire x1="137.16" y1="45.72" x2="137.16" y2="50.8" width="0.1524" layer="91"/>
+<label x="137.16" y="50.8" size="1.778" layer="95" rot="R90" xref="yes"/>
+</segment>
+</net>
