File: HW-MAPLE-Large/V4.0/AddOnSDuino/V4-AddOnSduino-V003.sch (EAGLE design)
At the start: 7 parts

Commit message: V4
Connections:
- removed net +3V3: CC1101.VCC
- net VCC: now also CC1101.VCC
Changed lines of the file:
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@@
 <part name="PORT20" library="frames" deviceset="PORT5" device=""/>
 <part name="PORT22" library="frames" deviceset="PORT5" device=""/>
-<part name="+3V3" library="supply1" deviceset="+3V3" device=""/>
 <part name="A11A" library="pinhead" deviceset="PINHD-1X1" device=""/>
 <part name="A11B" library="wireless" deviceset="SMA" device=""/>
@@
 <part name="PORT6" library="frames" deviceset="PORT7" device=""/>
 <part name="SUPPLY1" library="supply2" library_urn="urn:adsk.eagle:library:372" deviceset="VCC" device=""/>
+<part name="SUPPLY3" library="supply2" library_urn="urn:adsk.eagle:library:372" deviceset="VCC" device=""/>
 </parts>
 <sheets>
@@
 <instance part="PORT20" gate="G$1" x="-29.21" y="-127" smashed="yes" rot="R180"/>
 <instance part="PORT22" gate="G$1" x="-29.21" y="-139.7" smashed="yes" rot="R180"/>
-<instance part="+3V3" gate="G$1" x="-16.51" y="-111.76" smashed="yes">
-<attribute name="VALUE" x="-19.05" y="-116.84" size="1.778" layer="96" rot="R90"/>
-</instance>
 <instance part="A11A" gate="G$1" x="38.1" y="-149.86" smashed="yes">
 <attribute name="NAME" x="31.75" y="-146.685" size="1.778" layer="95"/>
@@
 <instance part="SUPPLY1" gate="G$1" x="33.02" y="-78.74" smashed="yes" rot="R270">
 <attribute name="VALUE" x="36.195" y="-76.835" size="1.778" layer="96" rot="R270"/>
+</instance>
+<instance part="SUPPLY3" gate="G$1" x="-20.32" y="-119.38" smashed="yes">
+<attribute name="VALUE" x="-22.225" y="-116.205" size="1.778" layer="96"/>
 </instance>
 </instances>
@@
 <wire x1="30.48" y1="-78.74" x2="25.4" y2="-78.74" width="0.1524" layer="91"/>
 </segment>
+<segment>
+<wire x1="-20.32" y1="-121.92" x2="-13.97" y2="-121.92" width="0.1524" layer="91"/>
+<pinref part="CC1101" gate="G$1" pin="VCC"/>
+<pinref part="SUPPLY3" gate="G$1" pin="VCC"/>
+</segment>
 </net>
 <net name="TX-MAPLE0" class="0">
@@
 </segment>
 </net>
-<net name="+3V3" class="0">
-<segment>
-<wire x1="-16.51" y1="-121.92" x2="-13.97" y2="-121.92" width="0.1524" layer="91"/>
-<wire x1="-16.51" y1="-121.92" x2="-16.51" y2="-114.3" width="0.1524" layer="91"/>
-<pinref part="+3V3" gate="G$1" pin="+3V3"/>
-<pinref part="CC1101" gate="G$1" pin="VCC"/>
-</segment>
-</net>
