File: HW-MAPLE-Large/V4.0/AddOnZigbeeSMD/V4-AddOnZigbee-SMD-V002.sch (EAGLE design)
At the start: 5 parts

Commit message: V4 Test
Parts:
- U$1: value CC2530CC2530PA -> CC2530; device zigbee:CC2530CC2530PA -> zigbee:CC2530
Changed lines of the file:
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@@
 <part name="SUPPLY10" library="supply2" library_urn="urn:adsk.eagle:library:372" deviceset="VCC" device=""/>
 <part name="GND15" library="supply1" library_urn="urn:adsk.eagle:library:371" deviceset="GND" device=""/>
-<part name="GND3" library="supply1" library_urn="urn:adsk.eagle:library:371" deviceset="GND" device=""/>
-<part name="SUPPLY3" library="supply2" library_urn="urn:adsk.eagle:library:372" deviceset="VCC" device=""/>
 <part name="CC-DEBUG" library="con-lstb" library_urn="urn:adsk.eagle:library:162" deviceset="MA05-2" device="" package3d_urn="urn:adsk.eagle:package:8329/1"/>
-<part name="U$1" library="zigbee" deviceset="CC2530" device="CC2530PA"/>
+<part name="U$1" library="zigbee" deviceset="CC2530" device="" value="CC2530"/>
 <part name="GND6" library="supply1" library_urn="urn:adsk.eagle:library:371" deviceset="GND" device=""/>
 <part name="SUPPLY7" library="supply2" library_urn="urn:adsk.eagle:library:372" deviceset="VCC" device=""/>
+<part name="GND2" library="supply1" library_urn="urn:adsk.eagle:library:371" deviceset="GND" device=""/>
+<part name="SUPPLY1" library="supply2" library_urn="urn:adsk.eagle:library:372" deviceset="VCC" device=""/>
 </parts>
 <sheets>
@@
 <attribute name="VALUE" x="242.57" y="-77.47" size="1.778" layer="96"/>
 </instance>
-<instance part="GND3" gate="1" x="116.84" y="-104.14" smashed="yes" rot="R180">
-<attribute name="VALUE" x="119.38" y="-101.6" size="1.778" layer="96" rot="R180"/>
-</instance>
-<instance part="SUPPLY3" gate="G$1" x="152.4" y="-121.92" smashed="yes" rot="R270">
-<attribute name="VALUE" x="155.575" y="-120.015" size="1.778" layer="96" rot="R270"/>
-</instance>
 <instance part="CC-DEBUG" gate="G$1" x="193.04" y="-111.76" smashed="yes" rot="R180">
 <attribute name="VALUE" x="196.85" y="-101.6" size="1.778" layer="96" rot="R180"/>
@@
 <instance part="SUPPLY7" gate="G$1" x="91.44" y="-203.2" smashed="yes" rot="R90">
 <attribute name="VALUE" x="88.265" y="-205.105" size="1.778" layer="96" rot="R90"/>
+</instance>
+<instance part="GND2" gate="1" x="91.44" y="-132.08" smashed="yes" rot="R270">
+<attribute name="VALUE" x="88.9" y="-129.54" size="1.778" layer="96" rot="R270"/>
+</instance>
+<instance part="SUPPLY1" gate="G$1" x="91.44" y="-139.7" smashed="yes" rot="R90">
+<attribute name="VALUE" x="88.265" y="-141.605" size="1.778" layer="96" rot="R90"/>
 </instance>
 </instances>
@@
 <pinref part="GND15" gate="1" pin="GND"/>
 <wire x1="245.11" y1="-71.12" x2="245.11" y2="-72.39" width="0.1524" layer="91"/>
-</segment>
-<segment>
-<pinref part="GND3" gate="1" pin="GND"/>
-<wire x1="116.84" y1="-106.68" x2="86.36" y2="-106.68" width="0.1524" layer="91"/>
-<wire x1="86.36" y1="-106.68" x2="86.36" y2="-116.84" width="0.1524" layer="91"/>
-<wire x1="86.36" y1="-116.84" x2="93.98" y2="-116.84" width="0.1524" layer="91"/>
-<wire x1="142.24" y1="-116.84" x2="149.86" y2="-116.84" width="0.1524" layer="91"/>
-<wire x1="149.86" y1="-116.84" x2="149.86" y2="-106.68" width="0.1524" layer="91"/>
-<wire x1="149.86" y1="-106.68" x2="116.84" y2="-106.68" width="0.1524" layer="91"/>
-<junction x="116.84" y="-106.68"/>
 </segment>
 <segment>
@@
 <wire x1="96.52" y1="-198.12" x2="101.6" y2="-198.12" width="0.1524" layer="91"/>
 <junction x="96.52" y="-195.58"/>
+</segment>
+<segment>
+<pinref part="GND2" gate="1" pin="GND"/>
+<wire x1="101.6" y1="-132.08" x2="96.52" y2="-132.08" width="0.1524" layer="91"/>
+<wire x1="96.52" y1="-132.08" x2="93.98" y2="-132.08" width="0.1524" layer="91"/>
+<wire x1="96.52" y1="-132.08" x2="96.52" y2="-134.62" width="0.1524" layer="91"/>
+<wire x1="96.52" y1="-134.62" x2="101.6" y2="-134.62" width="0.1524" layer="91"/>
+<junction x="96.52" y="-132.08"/>
 </segment>
 </net>
@@
 <junction x="96.52" y="-203.2"/>
 </segment>
+<segment>
+<pinref part="SUPPLY1" gate="G$1" pin="VCC"/>
+<wire x1="101.6" y1="-139.7" x2="96.52" y2="-139.7" width="0.1524" layer="91"/>
+<wire x1="96.52" y1="-139.7" x2="93.98" y2="-139.7" width="0.1524" layer="91"/>
+<wire x1="101.6" y1="-137.16" x2="96.52" y2="-137.16" width="0.1524" layer="91"/>
+<wire x1="96.52" y1="-137.16" x2="96.52" y2="-139.7" width="0.1524" layer="91"/>
+<junction x="96.52" y="-139.7"/>
+</segment>
 </net>
 <net name="RX0" class="0">
@@
 </segment>
 <segment>
-<wire x1="142.24" y1="-152.4" x2="160.02" y2="-152.4" width="0.1524" layer="91"/>
-<wire x1="160.02" y1="-152.4" x2="162.56" y2="-152.4" width="0.1524" layer="91"/>
-<label x="149.86" y="-152.4" size="1.778" layer="95"/>
-</segment>
-<segment>
 <pinref part="U$1" gate="G$1" pin="P0.3"/>
 <wire x1="132.08" y1="-205.74" x2="147.32" y2="-205.74" width="0.1524" layer="91"/>
 <label x="139.7" y="-205.74" size="1.778" layer="95"/>
+</segment>
+<segment>
+<wire x1="132.08" y1="-142.24" x2="147.32" y2="-142.24" width="0.1524" layer="91"/>
+<label x="139.7" y="-142.24" size="1.778" layer="95"/>
 </segment>
 </net>
@@
 </segment>
 <segment>
-<wire x1="142.24" y1="-147.32" x2="160.02" y2="-147.32" width="0.1524" layer="91"/>
-<label x="149.86" y="-147.32" size="1.778" layer="95"/>
-</segment>
-<segment>
 <pinref part="U$1" gate="G$1" pin="P0.2"/>
 <wire x1="132.08" y1="-203.2" x2="147.32" y2="-203.2" width="0.1524" layer="91"/>
 <label x="139.7" y="-203.2" size="1.778" layer="95"/>
 </segment>
+<segment>
+<wire x1="132.08" y1="-139.7" x2="147.32" y2="-139.7" width="0.1524" layer="91"/>
+<label x="139.7" y="-139.7" size="1.778" layer="95"/>
+</segment>
 </net>
 <net name="DC" class="0">
@@
 </segment>
 <segment>
-<wire x1="93.98" y1="-157.48" x2="73.66" y2="-157.48" width="0.1524" layer="91"/>
-<label x="76.2" y="-157.48" size="1.778" layer="95"/>
-</segment>
-<segment>
 <pinref part="U$1" gate="G$1" pin="P2.2"/>
 <wire x1="101.6" y1="-205.74" x2="81.28" y2="-205.74" width="0.1524" layer="91"/>
 <label x="81.28" y="-205.74" size="1.778" layer="95" rot="R180" xref="yes"/>
 </segment>
+<segment>
+<wire x1="101.6" y1="-142.24" x2="81.28" y2="-142.24" width="0.1524" layer="91"/>
+<label x="81.28" y="-142.24" size="1.778" layer="95" rot="R180" xref="yes"/>
+</segment>
 </net>
 <net name="CS" class="0">
@@
 </segment>
 <segment>
-<wire x1="142.24" y1="-132.08" x2="160.02" y2="-132.08" width="0.1524" layer="91"/>
-<label x="152.4" y="-132.08" size="1.778" layer="95"/>
-</segment>
-<segment>
 <pinref part="U$1" gate="G$1" pin="RESET_N"/>
 <wire x1="132.08" y1="-195.58" x2="147.32" y2="-195.58" width="0.1524" layer="91"/>
 <label x="139.7" y="-195.58" size="1.778" layer="95"/>
 </segment>
+<segment>
+<wire x1="132.08" y1="-132.08" x2="147.32" y2="-132.08" width="0.1524" layer="91"/>
+<label x="139.7" y="-132.08" size="1.778" layer="95"/>
+</segment>
 </net>
 <net name="DD" class="0">
@@
 </segment>
 <segment>
-<wire x1="93.98" y1="-127" x2="73.66" y2="-127" width="0.1524" layer="91"/>
-<label x="76.2" y="-127" size="1.778" layer="95"/>
-</segment>
-<segment>
 <pinref part="U$1" gate="G$1" pin="P2.1"/>
 <wire x1="101.6" y1="-208.28" x2="83.82" y2="-208.28" width="0.1524" layer="91"/>
 <label x="83.82" y="-208.28" size="1.778" layer="95" rot="R180" xref="yes"/>
 </segment>
+<segment>
+<wire x1="101.6" y1="-144.78" x2="83.82" y2="-144.78" width="0.1524" layer="91"/>
+<label x="83.82" y="-144.78" size="1.778" layer="95" rot="R180" xref="yes"/>
+</segment>
 </net>
 <net name="SCLK" class="0">
@@
 <label x="88.9" y="-210.82" size="1.778" layer="95" rot="R180" xref="yes"/>
 </segment>
-</net>
-<net name="N$2" class="1">
-<segment>
-<wire x1="147.32" y1="-121.92" x2="142.24" y2="-121.92" width="0.1524" layer="91"/>
-<wire x1="142.24" y1="-127" x2="147.32" y2="-127" width="0.1524" layer="91"/>
-<wire x1="147.32" y1="-127" x2="147.32" y2="-121.92" width="0.1524" layer="91"/>
+<segment>
+<wire x1="101.6" y1="-147.32" x2="88.9" y2="-147.32" width="0.1524" layer="91"/>
+<label x="88.9" y="-147.32" size="1.778" layer="95" rot="R180" xref="yes"/>
 </segment>
 </net>
@@
 </drawing>
 <compatibility>
+<note version="6.3" minversion="6.2.2" severity="warning">
+Since Version 6.2.2 text objects can contain more than one line,
+which will not be processed correctly with this version.
+</note>
 <note version="8.2" severity="warning">
 Since Version 8.2, EAGLE supports online libraries. The ids
@@
 packages will not be understood (or retained) with this version.
 </note>
+<note version="8.4" severity="warning">
+Since Version 8.4, EAGLE supports properties for SPICE simulation.
+Probes in schematics and SPICE mapping objects found in parts and library devices
+will not be understood with this version. Update EAGLE to the latest version
+for full support of SPICE simulation.
+</note>
 </compatibility>
