File: HW-MAPLE-Large/V4.0/AddOnArduino-RFMx/V4-MySensors-LoRa-V005.brd (EAGLE design)
At the start: 39 x 20 mm, 8 parts, among them U1 RFM69HCW

Commit message: V4
Routing:
- net GND: vias 4 -> 22
- added copper zone on layer 1, net GND
- added copper zone on layer 16, net GND
Changed lines of the file:
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@@
 <setting verticaltext="up"/>
 </settings>
-<grid distance="10" unitdist="mil" unit="mil" style="lines" multiple="1" display="yes" altdistance="5" altunitdist="mil" altunit="mil"/>
+<grid distance="25" unitdist="mil" unit="mil" style="lines" multiple="1" display="yes" altdistance="5" altunitdist="mil" altunit="mil"/>
 <layers>
 <layer number="1" name="Top" color="4" fill="1" visible="yes" active="yes"/>
@@
 <wire x1="39" y1="20" x2="0" y2="20" width="0" layer="20"/>
 <wire x1="0" y1="20" x2="0" y2="0" width="0" layer="20"/>
-<wire x1="-4" y1="19" x2="50" y2="19" width="0.1524" layer="48" style="shortdash"/>
-<wire x1="47" y1="22" x2="47" y2="-5" width="0.1524" layer="48" style="shortdash"/>
-<wire x1="0" y1="22" x2="0" y2="-5" width="0.1524" layer="48" style="shortdash"/>
-<wire x1="-5" y1="0" x2="51" y2="0" width="0.1524" layer="48" style="shortdash"/>
 </plain>
 <attributes>
@@
 <wire x1="8.255" y1="13.38" x2="8.255" y2="12.048990625" width="0.4572" layer="16"/>
 <wire x1="36.83" y1="18.542" x2="36.83" y2="16.128990625" width="0.4572" layer="1"/>
+<polygon width="0.1524" layer="1">
+<vertex x="1.27" y="1.27"/>
+<vertex x="1.27" y="19.05"/>
+<vertex x="38.1" y="19.05"/>
+<vertex x="38.1" y="1.27"/>
+</polygon>
+<polygon width="0.1524" layer="16">
+<vertex x="1.27" y="19.05"/>
+<vertex x="38.1" y="19.05"/>
+<vertex x="38.1" y="1.27"/>
+<vertex x="1.27" y="1.27"/>
+</polygon>
+<via x="11.43" y="17.78" extent="1-16" drill="0.35"/>
+<wire x1="12.970990625" y1="15.382" x2="11.43" y2="17.78" width="0" layer="19" extent="16-16"/>
+<via x="6.35" y="2.54" extent="1-16" drill="0.35"/>
+<via x="10.16" y="2.54" extent="1-16" drill="0.35"/>
+<via x="13.97" y="17.78" extent="1-16" drill="0.35"/>
+<via x="12.065" y="11.43" extent="1-16" drill="0.35"/>
+<via x="12.065" y="6.985" extent="1-16" drill="0.35"/>
+<via x="6.35" y="6.985" extent="1-16" drill="0.35"/>
+<via x="19.05" y="17.78" extent="1-16" drill="0.35"/>
+<via x="19.685" y="15.875" extent="1-16" drill="0.35"/>
+<via x="26.035" y="10.795" extent="1-16" drill="0.35"/>
+<via x="26.67" y="1.905" extent="1-16" drill="0.35"/>
+<via x="25.4" y="6.985" extent="1-16" drill="0.35"/>
+<via x="36.83" y="14.605" extent="1-16" drill="0.35"/>
+<via x="36.83" y="2.54" extent="1-16" drill="0.35"/>
+<via x="34.29" y="2.54" extent="1-16" drill="0.35"/>
+<via x="36.195" y="5.715" extent="1-16" drill="0.35"/>
+<via x="37.465" y="9.525" extent="1-16" drill="0.35"/>
+<via x="35.56" y="12.7" extent="1-16" drill="0.35"/>
 </signal>
 <signal name="VCC" class="1">
