File: HW-MAPLE-Large/V4.0/AddOnESP32/V4-AddOnESP32-V008-cc1101.sch (EAGLE design)
At the start: 24 parts, among them U2 RFM69HCW, U3 ESP-WROOM-32

Commit message: V4
Parts:
- removed ANT1: (no value), pinhead:PINHD-1X1
- removed AP2112: 3.3V, SparkFun-IC-Power:V_REG_AP2112K-3.3V
- removed C2, C6: 22pF, rcl:C-EUC0805
- removed C7: (no value), rcl:C-EUC1812
- removed JP1: JUMPER-SMT_2_NC_PASTE_NO-SILK, SparkFun-Jumpers:JUMPER-SMT_2_NC_PASTE_NO-SILK
- removed R1: 10k, rcl:R-EU_M0805
- removed R2: 1M, rcl:R-EU_M0805
- removed R3: 470K, rcl:R-EU_M0805
- removed R7: 100k, rcl:R-EU_M0805
- removed U$1: MAPLE-CUL-ADDON-V01, Martin-Communication-V4:MAPLE-CUL-ADDON-V01
- removed U2: RFM69HCW, doug:RFM69HCW
- removed UART0: (no value), con-lstb:MA04-1
Connections:
- removed net ANT1: ANT1.1, U2.ANT
- removed net IN++: R7.1
- removed net MAYBE_IO5: CC0.GDO2, JP1.2
- removed net N$12: AP2112.EN, R7.2
- removed net N$4: U2.DIO2
- removed net N$8: U2.DIO1
- removed net N$9: U2.RESET
- removed net UREG: AP2112.IN, R2.1
- net GND: no longer AP2112.GND, C2.1, C6.2, C7.1, R3.1, U2.GND_1, U2.GND_2, U2.GND_3, UART0.4
- net IO16: no longer U2.DIO0
- net IO17: no longer R1.1, U2.NSS
- net IO18: no longer U2.SCK
- net IO19: no longer U2.MISO
- net IO22: no longer R2.2, R3.2
- net IO23: no longer U2.MOSI
- net IO5: now also CC0.GDO2; no longer JP1.1
- net RX-MAPLE0: no longer UART0.3
- net TX-MAPLE0: no longer UART0.2
- net VCC: no longer AP2112.OUT, C2.2, C6.1, C7.2, R1.2, U2.3.3V, UART0.1
