File: HW-MAPLE-Large/V4.0/AddOnTemplate/V4-AddOnLeer-V001.sch (EAGLE design)
At the start: 5 parts

Commit message: V4
Parts:
- removed UART1: (no value), con-lstb:MA04-1
Connections:
- net GND: no longer UART1.4
- net RX-MAPLE0: no longer UART1.3
- net TX-MAPLE0: no longer UART1.2
- net VCC: no longer UART1.1
Other:
- moved on the sheet: C6
Changed lines of the file:
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@@
 <part name="GND15" library="supply1" library_urn="urn:adsk.eagle:library:371" deviceset="GND" device=""/>
 <part name="U$1" library="Martin-Communication-V4" deviceset="MAPLE-CUL-ADDON-V01" device=""/>
-<part name="UART1" library="con-lstb" library_urn="urn:adsk.eagle:library:162" deviceset="MA04-1" device="" package3d_urn="urn:adsk.eagle:package:8337/1"/>
-<part name="GND2" library="supply1" library_urn="urn:adsk.eagle:library:371" deviceset="GND" device=""/>
-<part name="SUPPLY1" library="supply2" library_urn="urn:adsk.eagle:library:372" deviceset="VCC" device=""/>
 </parts>
 <sheets>
@@
 <attribute name="NAME" x="194.31" y="-156.972" size="1.778" layer="95" rot="R180"/>
 </instance>
-<instance part="GND1" gate="1" x="121.92" y="-30.48" smashed="yes" rot="R90">
-<attribute name="VALUE" x="124.46" y="-33.02" size="1.778" layer="96" rot="R90"/>
+<instance part="GND1" gate="1" x="231.14" y="-76.2" smashed="yes">
+<attribute name="VALUE" x="228.6" y="-78.74" size="1.778" layer="96"/>
 </instance>
 <instance part="GND7" gate="1" x="184.15" y="-158.75" smashed="yes">
@@
 <attribute name="VALUE" x="182.245" y="-137.795" size="1.778" layer="96"/>
 </instance>
-<instance part="C6" gate="G$1" x="101.6" y="-30.48" smashed="yes" rot="R90">
-<attribute name="NAME" x="101.219" y="-28.956" size="1.778" layer="95" rot="R90"/>
-<attribute name="VALUE" x="106.299" y="-28.956" size="1.778" layer="96" rot="R90"/>
+<instance part="C6" gate="G$1" x="231.14" y="-63.5" smashed="yes">
+<attribute name="NAME" x="232.664" y="-63.119" size="1.778" layer="95"/>
+<attribute name="VALUE" x="232.664" y="-68.199" size="1.778" layer="96"/>
 </instance>
-<instance part="SUPPLY2" gate="G$1" x="91.44" y="-30.48" smashed="yes" rot="R90">
-<attribute name="VALUE" x="88.265" y="-32.385" size="1.778" layer="96" rot="R90"/>
+<instance part="SUPPLY2" gate="G$1" x="231.14" y="-55.88" smashed="yes">
+<attribute name="VALUE" x="229.235" y="-52.705" size="1.778" layer="96"/>
 </instance>
 <instance part="C7" gate="G$1" x="248.92" y="-66.04" smashed="yes" rot="R180">
@@
 </instance>
 <instance part="U$1" gate="G$1" x="154.94" y="-71.12" smashed="yes"/>
-<instance part="UART1" gate="1" x="193.04" y="-186.69" smashed="yes" rot="R180">
-<attribute name="VALUE" x="194.31" y="-176.53" size="1.778" layer="96" rot="R180"/>
-<attribute name="NAME" x="194.31" y="-192.532" size="1.778" layer="95" rot="R180"/>
-</instance>
-<instance part="GND2" gate="1" x="184.15" y="-194.31" smashed="yes">
-<attribute name="VALUE" x="181.61" y="-196.85" size="1.778" layer="96"/>
-</instance>
-<instance part="SUPPLY1" gate="G$1" x="184.15" y="-176.53" smashed="yes">
-<attribute name="VALUE" x="182.245" y="-173.355" size="1.778" layer="96"/>
-</instance>
 </instances>
 <busses>
@@
 <pinref part="C6" gate="G$1" pin="2"/>
 <pinref part="GND1" gate="1" pin="GND"/>
-<wire x1="106.68" y1="-30.48" x2="119.38" y2="-30.48" width="0.1524" layer="91"/>
+<wire x1="231.14" y1="-68.58" x2="231.14" y2="-73.66" width="0.1524" layer="91"/>
 </segment>
 <segment>
@@
 <pinref part="GND15" gate="1" pin="GND"/>
 <wire x1="245.11" y1="-71.12" x2="245.11" y2="-72.39" width="0.1524" layer="91"/>
-</segment>
-<segment>
-<pinref part="GND2" gate="1" pin="GND"/>
-<wire x1="185.42" y1="-189.23" x2="184.15" y2="-189.23" width="0.1524" layer="91"/>
-<wire x1="184.15" y1="-189.23" x2="184.15" y2="-191.77" width="0.1524" layer="91"/>
-<pinref part="UART1" gate="1" pin="4"/>
 </segment>
 </net>
@@
 <pinref part="C6" gate="G$1" pin="1"/>
 <pinref part="SUPPLY2" gate="G$1" pin="VCC"/>
-<wire x1="99.06" y1="-30.48" x2="93.98" y2="-30.48" width="0.1524" layer="91"/>
+<wire x1="231.14" y1="-60.96" x2="231.14" y2="-58.42" width="0.1524" layer="91"/>
 </segment>
 <segment>
@@
 <wire x1="248.92" y1="-60.96" x2="248.92" y2="-58.42" width="0.1524" layer="91"/>
 <pinref part="SUPPLY10" gate="G$1" pin="VCC"/>
-</segment>
-<segment>
-<pinref part="SUPPLY1" gate="G$1" pin="VCC"/>
-<wire x1="185.42" y1="-181.61" x2="184.15" y2="-181.61" width="0.1524" layer="91"/>
-<wire x1="184.15" y1="-181.61" x2="184.15" y2="-179.07" width="0.1524" layer="91"/>
-<pinref part="UART1" gate="1" pin="1"/>
 </segment>
 </net>
@@
 <label x="172.72" y="-148.59" size="1.778" layer="95"/>
 <pinref part="UART0" gate="1" pin="2"/>
-</segment>
-<segment>
-<wire x1="185.42" y1="-184.15" x2="173.99" y2="-184.15" width="0.1524" layer="91"/>
-<wire x1="173.99" y1="-184.15" x2="166.37" y2="-184.15" width="0.1524" layer="91"/>
-<label x="172.72" y="-184.15" size="1.778" layer="95"/>
-<pinref part="UART1" gate="1" pin="2"/>
 </segment>
 </net>
@@
 <label x="172.72" y="-151.13" size="1.778" layer="95"/>
 <pinref part="UART0" gate="1" pin="3"/>
-</segment>
-<segment>
-<wire x1="165.1" y1="-186.69" x2="172.72" y2="-186.69" width="0.1524" layer="91"/>
-<wire x1="172.72" y1="-186.69" x2="185.42" y2="-186.69" width="0.1524" layer="91"/>
-<label x="172.72" y="-186.69" size="1.778" layer="95"/>
-<pinref part="UART1" gate="1" pin="3"/>
 </segment>
 </net>
@@
 packages will not be understood (or retained) with this version.
 </note>
+<note version="8.4" severity="warning">
+Since Version 8.4, EAGLE supports properties for SPICE simulation.
+Probes in schematics and SPICE mapping objects found in parts and library devices
+will not be understood with this version. Update EAGLE to the latest version
+for full support of SPICE simulation.
+</note>
 </compatibility>
