File: HW-MAPLE-Large/V4.0/AddOnCC1101/V4-AddOnSduino-V02-008.sch (EAGLE design)
At the start: 8 parts, among them U1 RFM69HCW

Commit message: V4 General Update
Parts:
- removed ANT1: (no value), pinhead:PINHD-1X1
- removed U1: RFM69HCW, doug:RFM69HCW
- removed UART0: (no value), con-lstb:MA04-1
- removed X2: (no value), adafruit:SMACONNECTOR_EDGE
- added A11A: (no value), pinhead:PINHD-1X1
- added A11B: SMA, wireless:SMA
- added CC1101: CC1101_MODULE1SMD, CC1101:CC1101_MODULE1SMD
- added U$2: MAPLE-CUL-ADDON-V01, Martin-Communication-V4:MAPLE-CUL-ADDON-V01
Connections:
- removed net ANT1: ANT1.1, U1.ANT, X2.ANT
- removed net N$14: U1.DIO2
- removed net N$15: U1.DIO1
- removed net N$2: U$1.RX1, UART0.2
- removed net N$3: U1.RESET
- removed net RX-MAPLE0: U$1.TX0, UART0.3
- new net ANT2: A11A.1, A11B.1, CC1101.ANT
- new net CSN: CC1101.CSN, R2.1
- new net GDO0_D3: CC1101.GDO0
- new net GDO2_D2: CC1101.GDO2
- new net MISO: CC1101.MISO
- new net MOSI: CC1101.MOSI
- new net RX0: U$1.TX0, U$2.TX-MAPLE
- new net SCK: CC1101.SCLK
- new net TX0: U$1.RX1, U$2.RX-MAPLE
- net CSN-A: no longer R2.1, U1.NSS
- net GND: now also A11B.2, A11B.3, A11B.4, A11B.5, CC1101.GND@1, CC1101.GND@2, CC1101.GND@3, U$2.GND, U$2.GND1; no longer U1.GND_1, U1.GND_2, U1.GND_3, UART0.4, X2.GND1, X2.GND2, X2.GND3, X2.GND4
- net IRQ-A: no longer U1.DIO0
- net MISO-A: no longer U1.MISO
- net MOSI-A: no longer U1.MOSI
- net SCK-A: no longer U1.SCK
- net VCC: now also CC1101.VCC, U$2.VCC, U$2.VCC1; no longer U1.3.3V, UART0.1
Other:
- moved on the sheet: R2
