File: HW-MAPLE-Large/V4.0/AddOnCC1101/V4-AddOnSduino-V02-009.sch (EAGLE design)
At the start: 7 parts

Commit message: V4 General Update
Parts:
- removed UART0: (no value), con-lstb:MA04-1
- added R2: 10k, rcl:R-EU_M0805
- added U$1: MARTIN-PROMINI-SPI, Arduino-clone:MARTIN-PROMINI-SPI
- U$2: value MARTIN-PROMINI-CC1101 -> MAPLE-CUL-ADDON-V01; device Arduino-clone:MARTIN-PROMINI-CC1101 -> Martin-Communication-V4:MAPLE-CUL-ADDON-V01
Connections:
- net ANT1 renamed ANT2
- removed net RX-MAPLE0: U$2.TX0, UART0.3
- removed net TX-MAPLE0: U$2.RX1, UART0.2
- new net CSN-A: U$1.D10
- new net IRQ-A: U$1.D2
- new net MISO-A: U$1.D12
- new net MOSI-A: U$1.D11
- new net N$11: U$1.RAW
- new net N$9: U$1.RST
- new net RX0: U$1.RX1, U$2.TX-MAPLE
- new net SCK-A: U$1.D13
- new net TX0: U$1.TX0, U$2.RX-MAPLE
- net CSN: now also R2.1; no longer U$2.D10
- net GDO0_D3: no longer U$2.D3
- net GDO2_D2: no longer U$2.D2
- net GND: now also U$1.GND, U$2.GND1; no longer UART0.4
- net MISO: no longer U$2.D12
- net MOSI: no longer U$2.D11
- net SCK: no longer U$2.D13
- net VCC: now also R2.2, U$1.VCC, U$2.VCC1; no longer UART0.1
Other:
- moved on the sheet: A11A, A11B, C6, C7, CC1101
