File: HW-MAPLE-Large/V4.0/AddOn-RS485/V4-AddRS485-1W-V01-016-defect.sch (EAGLE design)
At the start: 16 parts, among them X1 1751248, X7 1751264

Commit message: V4-AddOns ; Large
Parts:
- removed 5V: JUMPER-SMT_2_NC_PASTE_NO-SILK, SparkFun-Jumpers:JUMPER-SMT_2_NC_PASTE_NO-SILK
- added 1W, GND7: (no value), jumper:SJ
- added IC2: DS2480B, 1wire:DS2480B
- added Q2: BSS123, transistor-small-signal:BSS123
- added R1, R3: 4k7, rcl:R-EU_R0805
- added R2: 10k, rcl:R-EU_R0805
- added ZD2: DS9503P, 1wire:DS9503P
Connections:
- net IN renamed EXTIN
- removed net VCC-: JP2.1, U$3.VCC
- new net N$1: C10.2, JP1.2
- new net N$3: IC2.1W, ZD2.P$4
- new net N$4: GND7.2, X7-4.K, ZD2.P$2
- new net N$6: Q2.G, R1.2, R2.1
- new net RX1: IC2.TXD
- new net TX1: IC2.RXD
- net 1W: now also 1W.1, Q2.S, ZD2.P$1
- net 5V: now also R1.1, R3.1; no longer 5V.2
- net A: now also 1W.2, JP2.1, JP2.2, Q2.D, R3.2
- net GND: now also GND7.1, IC2.GND, J2-1.S1, J2-1.S2, R2.2, ZD2.P$3; no longer X7-4.K
- net N$13: no longer 5V.1
- net V-RS485: now also IC2.POL, IC2.VDD, IC2.VPP; no longer C10.2, JP1.2
- net VCC: now also U$3.VCC; no longer JP2.2
Other:
- note added: "OneWire (or RS485 Connections)"
- moved on the sheet: C10, JP1, JP2
